Commit message: Added code to measure distance from origin

File: parserTest.urdf (robot description, URDF)
Before this commit: robot paul, 8 links, 7 joints
Links:
- removed link 09821ecb
- removed link 171d9b21
- removed link 3837421a
- removed link 6023bef8
- removed link 60c70f33
- removed link 8f60c46e
- removed link ce10f7fe
- removed link cf1ff730
- added link 1d5aa4d5, mass 1; collision box size=0.2 0.2 0.2; visual box size=0.2 0.2 0.2
- added link 367ebd77, mass 1; collision box size=0.2 0.2 0.2; visual box size=0.2 0.2 0.2
- added link 4fa08bce, mass 1; collision box size=0.2 0.2 0.2; visual box size=0.2 0.2 0.2
- added link 51242e42, mass 1; collision box size=0.2 0.2 0.2; visual box size=0.2 0.2 0.2
- added link d3199206, mass 1; collision box size=0.2 0.2 0.2; visual box size=0.2 0.2 0.2
- added link e143bdb5, mass 1; collision box size=0.2 0.2 0.2; visual box size=0.2 0.2 0.2
- added link f824428a, mass 1; collision box size=0.2 0.2 0.2; visual box size=0.2 0.2 0.2
- added link fadabb44, mass 1; collision box size=0.2 0.2 0.2; visual box size=0.2 0.2 0.2
Joints:
- removed joint 09821ecb171d9b21
- removed joint 171d9b2160c70f33
- removed joint 60c70f33ce10f7fe
- removed joint 60c70f33cf1ff730
- removed joint 8f60c46e09821ecb
- removed joint ce10f7fe3837421a
- removed joint ce10f7fe6023bef8
- added joint 51242e42e143bdb5: type revolute, parent 51242e42, child e143bdb5, origin xyz=0 0.2 0 rpy=0 0 0, axis 0 0 1, limit lower=-1.9 upper=1.9 effort=0 velocity=0
- added joint d319920651242e42: type revolute, parent d3199206, child 51242e42, origin xyz=0 0.2 0 rpy=0 0 0, axis 0 0 1, limit lower=-1.9 upper=1.9 effort=0 velocity=0
- added joint e143bdb5fadabb44: type revolute, parent e143bdb5, child fadabb44, origin xyz=0 0.2 0 rpy=0 0 0, axis 0 0 1, limit lower=-1.9 upper=1.9 effort=0 velocity=0
- added joint f824428a1d5aa4d5: type revolute, parent f824428a, child 1d5aa4d5, origin xyz=0 -0.2 0 rpy=0 0 0, axis 0 0 1, limit lower=-1.9 upper=1.9 effort=0 velocity=0
- added joint f824428a4fa08bce: type revolute, parent f824428a, child 4fa08bce, origin xyz=0 0 0.2 rpy=0 0 0, axis 0 0 1, limit lower=-1.9 upper=1.9 effort=0 velocity=0
- added joint fadabb44367ebd77: type revolute, parent fadabb44, child 367ebd77, origin xyz=0 0.2 0 rpy=0 0 0, axis 0 0 1, limit lower=-1.9 upper=1.9 effort=0 velocity=0
- added joint fadabb44f824428a: type revolute, parent fadabb44, child f824428a, origin xyz=-0.2 0 0 rpy=0 0 0, axis 0 0 1, limit lower=-1.9 upper=1.9 effort=0 velocity=0

Commit message: Added rudimentary generator script

File: parserTest.urdf (robot description, URDF)
Before this commit: robot paul, 8 links, 7 joints
Links:
- removed link 1d5aa4d5
- removed link 367ebd77
- removed link 4fa08bce
- removed link 51242e42
- removed link d3199206
- removed link e143bdb5
- removed link f824428a
- removed link fadabb44
- added link 19a95b51, mass 1; collision box size=0.2 0.2 0.2; visual box size=0.2 0.2 0.2
- added link 1ba917cd, mass 1; collision box size=0.2 0.2 0.2; visual box size=0.2 0.2 0.2
- added link 1f5d8327, mass 1; collision box size=0.2 0.2 0.2; visual box size=0.2 0.2 0.2
- added link 2427c4e1, mass 1; collision box size=0.2 0.2 0.2; visual box size=0.2 0.2 0.2
- added link 30be046c, mass 1; collision box size=0.2 0.2 0.2; visual box size=0.2 0.2 0.2
- added link 58d579ee, mass 1; collision box size=0.2 0.2 0.2; visual box size=0.2 0.2 0.2
- added link 5cc1c2c2, mass 1; collision box size=0.2 0.2 0.2; visual box size=0.2 0.2 0.2
- added link 5cdf790f, mass 1; collision box size=0.2 0.2 0.2; visual box size=0.2 0.2 0.2
- added link 6485ace6, mass 1; collision box size=0.2 0.2 0.2; visual box size=0.2 0.2 0.2
- added link 83c1f939, mass 1; collision box size=0.2 0.2 0.2; visual box size=0.2 0.2 0.2
- added link 8bf8317a, mass 1; collision box size=0.2 0.2 0.2; visual box size=0.2 0.2 0.2
- added link 9a8e9899, mass 1; collision box size=0.2 0.2 0.2; visual box size=0.2 0.2 0.2
- added link a012ceca, mass 1; collision box size=0.2 0.2 0.2; visual box size=0.2 0.2 0.2
- added link a7e97cdd, mass 1; collision box size=0.2 0.2 0.2; visual box size=0.2 0.2 0.2
- added link af362fe3, mass 1; collision box size=0.2 0.2 0.2; visual box size=0.2 0.2 0.2
- added link ba02d405, mass 1; collision box size=0.2 0.2 0.2; visual box size=0.2 0.2 0.2
- added link bc62b5e3, mass 1; collision box size=0.2 0.2 0.2; visual box size=0.2 0.2 0.2
- added link d7a25923, mass 1; collision box size=0.2 0.2 0.2; visual box size=0.2 0.2 0.2
- added link f13a5d97, mass 1; collision box size=0.2 0.2 0.2; visual box size=0.2 0.2 0.2
Joints:
- removed joint 51242e42e143bdb5
- removed joint d319920651242e42
- removed joint e143bdb5fadabb44
- removed joint f824428a1d5aa4d5
- removed joint f824428a4fa08bce
- removed joint fadabb44367ebd77
- removed joint fadabb44f824428a
- added joint 19a95b515cc1c2c2: type revolute, parent 19a95b51, child 5cc1c2c2, origin xyz=0 0.2 0 rpy=0 0 0, axis 0 0 1, limit lower=-1.9 upper=1.9 effort=0 velocity=0
- added joint 1ba917cd30be046c: type revolute, parent 1ba917cd, child 30be046c, origin xyz=0 0.2 0 rpy=0 0 0, axis 0 0 1, limit lower=-1.9 upper=1.9 effort=0 velocity=0
- added joint 5cc1c2c21ba917cd: type revolute, parent 5cc1c2c2, child 1ba917cd, origin xyz=0 0.2 0 rpy=0 0 0, axis 0 0 1, limit lower=-1.9 upper=1.9 effort=0 velocity=0
- added joint 5cdf790f1f5d8327: type revolute, parent 5cdf790f, child 1f5d8327, origin xyz=0 -0.2 0 rpy=0 0 0, axis 0 0 1, limit lower=-1.9 upper=1.9 effort=0 velocity=0
- added joint 5cdf790f83c1f939: type revolute, parent 5cdf790f, child 83c1f939, origin xyz=0 0.2 0 rpy=0 0 0, axis 0 0 1, limit lower=-1.9 upper=1.9 effort=0 velocity=0
- added joint 5cdf790faf362fe3: type revolute, parent 5cdf790f, child af362fe3, origin xyz=-0.2 0 0 rpy=0 0 0, axis 0 0 1, limit lower=-1.9 upper=1.9 effort=0 velocity=0
- added joint 8bf8317abc62b5e3: type revolute, parent 8bf8317a, child bc62b5e3, origin xyz=0 0.2 0 rpy=0 0 0, axis 0 0 1, limit lower=-1.9 upper=1.9 effort=0 velocity=0
- added joint 9a8e9899a7e97cdd: type revolute, parent 9a8e9899, child a7e97cdd, origin xyz=0 0.2 0 rpy=0 0 0, axis 0 0 1, limit lower=-1.9 upper=1.9 effort=0 velocity=0
- added joint a012cecad7a25923: type revolute, parent a012ceca, child d7a25923, origin xyz=0 0.2 0 rpy=0 0 0, axis 0 0 1, limit lower=-1.9 upper=1.9 effort=0 velocity=0
- added joint a7e97cdda012ceca: type revolute, parent a7e97cdd, child a012ceca, origin xyz=0.2 0 0 rpy=0 0 0, axis 0 0 1, limit lower=-1.9 upper=1.9 effort=0 velocity=0
- added joint af362fe32427c4e1: type revolute, parent af362fe3, child 2427c4e1, origin xyz=0 0.2 0 rpy=0 0 0, axis 0 0 1, limit lower=-1.9 upper=1.9 effort=0 velocity=0
- added joint af362fe358d579ee: type revolute, parent af362fe3, child 58d579ee, origin xyz=0.2 0 0 rpy=0 0 0, axis 0 0 1, limit lower=-1.9 upper=1.9 effort=0 velocity=0
- added joint af362fe39a8e9899: type revolute, parent af362fe3, child 9a8e9899, origin xyz=0 -0.2 0 rpy=0 0 0, axis 0 0 1, limit lower=-1.9 upper=1.9 effort=0 velocity=0
- added joint ba02d405f13a5d97: type revolute, parent ba02d405, child f13a5d97, origin xyz=0 0.2 0 rpy=0 0 0, axis 0 0 1, limit lower=-1.9 upper=1.9 effort=0 velocity=0
- added joint bc62b5e35cdf790f: type revolute, parent bc62b5e3, child 5cdf790f, origin xyz=0 0.2 0 rpy=0 0 0, axis 0 0 1, limit lower=-1.9 upper=1.9 effort=0 velocity=0
- added joint d7a25923ba02d405: type revolute, parent d7a25923, child ba02d405, origin xyz=0 0.2 0 rpy=0 0 0, axis 0 0 1, limit lower=-1.9 upper=1.9 effort=0 velocity=0
- added joint f13a5d9719a95b51: type revolute, parent f13a5d97, child 19a95b51, origin xyz=0.2 0 0 rpy=0 0 0, axis 0 0 1, limit lower=-1.9 upper=1.9 effort=0 velocity=0
- added joint f13a5d976485ace6: type revolute, parent f13a5d97, child 6485ace6, origin xyz=0 0.2 0 rpy=0 0 0, axis 0 0 1, limit lower=-1.9 upper=1.9 effort=0 velocity=0

Commit message: added Main.py to evaluate generations in batches

File: parserTest.urdf (robot description, URDF)
Before this commit: robot paul, 19 links, 18 joints
Links:
- removed link 19a95b51
- removed link 1ba917cd
- removed link 1f5d8327
- removed link 2427c4e1
- removed link 30be046c
- removed link 58d579ee
- removed link 5cc1c2c2
- removed link 5cdf790f
- removed link 6485ace6
- removed link 83c1f939
- removed link 8bf8317a
- removed link 9a8e9899
- removed link a012ceca
- removed link a7e97cdd
- removed link af362fe3
- removed link ba02d405
- removed link bc62b5e3
- removed link d7a25923
- removed link f13a5d97
- added link 0231e818, mass 1; collision box size=0.2 0.2 0.2; visual box size=0.2 0.2 0.2
- added link 0dc9647a, mass 1; collision box size=0.2 0.2 0.2; visual box size=0.2 0.2 0.2
- added link 0fd258d7, mass 1; collision box size=0.2 0.2 0.2; visual box size=0.2 0.2 0.2
- added link 1234c791, mass 1; collision box size=0.2 0.2 0.2; visual box size=0.2 0.2 0.2
- added link 1511502a, mass 1; collision box size=0.2 0.2 0.2; visual box size=0.2 0.2 0.2
- added link 181f7e2d, mass 1; collision box size=0.2 0.2 0.2; visual box size=0.2 0.2 0.2
- added link 23d9b26f, mass 1; collision box size=0.2 0.2 0.2; visual box size=0.2 0.2 0.2
- added link 24b6d36c, mass 1; collision box size=0.2 0.2 0.2; visual box size=0.2 0.2 0.2
- added link 2fdbc30e, mass 1; collision box size=0.2 0.2 0.2; visual box size=0.2 0.2 0.2
- added link 31b12c7b, mass 1; collision box size=0.2 0.2 0.2; visual box size=0.2 0.2 0.2
- added link 31c6b757, mass 1; collision box size=0.2 0.2 0.2; visual box size=0.2 0.2 0.2
- added link 38092bac, mass 1; collision box size=0.2 0.2 0.2; visual box size=0.2 0.2 0.2
- added link 3a06f8cc, mass 1; collision box size=0.2 0.2 0.2; visual box size=0.2 0.2 0.2
- added link 434e5162, mass 1; collision box size=0.2 0.2 0.2; visual box size=0.2 0.2 0.2
- added link 43be07d9, mass 1; collision box size=0.2 0.2 0.2; visual box size=0.2 0.2 0.2
- added link 45cbe0e2, mass 1; collision box size=0.2 0.2 0.2; visual box size=0.2 0.2 0.2
- added link 5392b5b2, mass 1; collision box size=0.2 0.2 0.2; visual box size=0.2 0.2 0.2
- added link 581c2250, mass 1; collision box size=0.2 0.2 0.2; visual box size=0.2 0.2 0.2
- added link 62d6a4e2, mass 1; collision box size=0.2 0.2 0.2; visual box size=0.2 0.2 0.2
- added link 63bd3236, mass 1; collision box size=0.2 0.2 0.2; visual box size=0.2 0.2 0.2
- added link 662e1da3, mass 1; collision box size=0.2 0.2 0.2; visual box size=0.2 0.2 0.2
- added link 6722bfd0, mass 1; collision box size=0.2 0.2 0.2; visual box size=0.2 0.2 0.2
- added link 68c0e889, mass 1; collision box size=0.2 0.2 0.2; visual box size=0.2 0.2 0.2
- added link 7187bc4c, mass 1; collision box size=0.2 0.2 0.2; visual box size=0.2 0.2 0.2
- added link 73436589, mass 1; collision box size=0.2 0.2 0.2; visual box size=0.2 0.2 0.2
- added link 84c3bc2a, mass 1; collision box size=0.2 0.2 0.2; visual box size=0.2 0.2 0.2
- added link 87d6d9a5, mass 1; collision box size=0.2 0.2 0.2; visual box size=0.2 0.2 0.2
- added link 935073ed, mass 1; collision box size=0.2 0.2 0.2; visual box size=0.2 0.2 0.2
- added link 9c2da2f4, mass 1; collision box size=0.2 0.2 0.2; visual box size=0.2 0.2 0.2
- added link 9ec0e600, mass 1; collision box size=0.2 0.2 0.2; visual box size=0.2 0.2 0.2
- added link a7ead54c, mass 1; collision box size=0.2 0.2 0.2; visual box size=0.2 0.2 0.2
- added link a8351408, mass 1; collision box size=0.2 0.2 0.2; visual box size=0.2 0.2 0.2
- added link ac6cf6e8, mass 1; collision box size=0.2 0.2 0.2; visual box size=0.2 0.2 0.2
- added link ad8c639e, mass 1; collision box size=0.2 0.2 0.2; visual box size=0.2 0.2 0.2
- added link adb2dd0f, mass 1; collision box size=0.2 0.2 0.2; visual box size=0.2 0.2 0.2
- added link b066414d, mass 1; collision box size=0.2 0.2 0.2; visual box size=0.2 0.2 0.2
- added link b3ea44e5, mass 1; collision box size=0.2 0.2 0.2; visual box size=0.2 0.2 0.2
- added link b7a98a4a, mass 1; collision box size=0.2 0.2 0.2; visual box size=0.2 0.2 0.2
- added link bc24cd03, mass 1; collision box size=0.2 0.2 0.2; visual box size=0.2 0.2 0.2
- added link bcc4c2ba, mass 1; collision box size=0.2 0.2 0.2; visual box size=0.2 0.2 0.2
- added link c0a43814, mass 1; collision box size=0.2 0.2 0.2; visual box size=0.2 0.2 0.2
- added link c209a4f2, mass 1; collision box size=0.2 0.2 0.2; visual box size=0.2 0.2 0.2
- added link cd08ca72, mass 1; collision box size=0.2 0.2 0.2; visual box size=0.2 0.2 0.2
- added link d0ee7787, mass 1; collision box size=0.2 0.2 0.2; visual box size=0.2 0.2 0.2
- added link d1ea9a80, mass 1; collision box size=0.2 0.2 0.2; visual box size=0.2 0.2 0.2
- added link d7336e02, mass 1; collision box size=0.2 0.2 0.2; visual box size=0.2 0.2 0.2
- added link d779f3c3, mass 1; collision box size=0.2 0.2 0.2; visual box size=0.2 0.2 0.2
- added link dc94f799, mass 1; collision box size=0.2 0.2 0.2; visual box size=0.2 0.2 0.2
- added link e400f108, mass 1; collision box size=0.2 0.2 0.2; visual box size=0.2 0.2 0.2
- added link f35b71d8, mass 1; collision box size=0.2 0.2 0.2; visual box size=0.2 0.2 0.2
- added link f49de8b1, mass 1; collision box size=0.2 0.2 0.2; visual box size=0.2 0.2 0.2
- added link f6724a8b, mass 1; collision box size=0.2 0.2 0.2; visual box size=0.2 0.2 0.2
- added link f8367eb9, mass 1; collision box size=0.2 0.2 0.2; visual box size=0.2 0.2 0.2
- added link ff371f0e, mass 1; collision box size=0.2 0.2 0.2; visual box size=0.2 0.2 0.2
Joints:
- removed joint 19a95b515cc1c2c2
- removed joint 1ba917cd30be046c
- removed joint 5cc1c2c21ba917cd
- removed joint 5cdf790f1f5d8327
- removed joint 5cdf790f83c1f939
- removed joint 5cdf790faf362fe3
- removed joint 8bf8317abc62b5e3
- removed joint 9a8e9899a7e97cdd
- removed joint a012cecad7a25923
- removed joint a7e97cdda012ceca
- removed joint af362fe32427c4e1
- removed joint af362fe358d579ee
- removed joint af362fe39a8e9899
- removed joint ba02d405f13a5d97
- removed joint bc62b5e35cdf790f
- removed joint d7a25923ba02d405
- removed joint f13a5d9719a95b51
- removed joint f13a5d976485ace6
- added joint 0dc9647a0231e818: type revolute, parent 0dc9647a, child 0231e818, origin xyz=0 0.2 0 rpy=0 0 0, axis 0 0 1, limit lower=-1.9 upper=1.9 effort=0 velocity=0
- added joint 1234c791434e5162: type revolute, parent 1234c791, child 434e5162, origin xyz=0 0.2 0 rpy=0 0 0, axis 0 0 1, limit lower=-1.9 upper=1.9 effort=0 velocity=0
- added joint 181f7e2d7187bc4c: type revolute, parent 181f7e2d, child 7187bc4c, origin xyz=0.2 0 0 rpy=0 0 0, axis 0 0 1, limit lower=-1.9 upper=1.9 effort=0 velocity=0
- added joint 23d9b26ff8367eb9: type revolute, parent 23d9b26f, child f8367eb9, origin xyz=0 0.2 0 rpy=0 0 0, axis 0 0 1, limit lower=-1.9 upper=1.9 effort=0 velocity=0
- added joint 24b6d36c31b12c7b: type revolute, parent 24b6d36c, child 31b12c7b, origin xyz=0 0.2 0 rpy=0 0 0, axis 0 0 1, limit lower=-1.9 upper=1.9 effort=0 velocity=0
- added joint 2fdbc30e45cbe0e2: type revolute, parent 2fdbc30e, child 45cbe0e2, origin xyz=0 0.2 0 rpy=0 0 0, axis 0 0 1, limit lower=-1.9 upper=1.9 effort=0 velocity=0
- added joint 31b12c7b581c2250: type revolute, parent 31b12c7b, child 581c2250, origin xyz=0.2 0 0 rpy=0 0 0, axis 0 0 1, limit lower=-1.9 upper=1.9 effort=0 velocity=0
- added joint 31c6b75723d9b26f: type revolute, parent 31c6b757, child 23d9b26f, origin xyz=0 0.2 0 rpy=0 0 0, axis 0 0 1, limit lower=-1.9 upper=1.9 effort=0 velocity=0
- added joint 31c6b757ad8c639e: type revolute, parent 31c6b757, child ad8c639e, origin xyz=0 0.2 0 rpy=0 0 0, axis 0 0 1, limit lower=-1.9 upper=1.9 effort=0 velocity=0
- added joint 38092bac0fd258d7: type revolute, parent 38092bac, child 0fd258d7, origin xyz=0 0.2 0 rpy=0 0 0, axis 0 0 1, limit lower=-1.9 upper=1.9 effort=0 velocity=0
- added joint 434e5162a8351408: type revolute, parent 434e5162, child a8351408, origin xyz=0 0.2 0 rpy=0 0 0, axis 0 0 1, limit lower=-1.9 upper=1.9 effort=0 velocity=0
- added joint 45cbe0e26722bfd0: type revolute, parent 45cbe0e2, child 6722bfd0, origin xyz=0 0.2 0 rpy=0 0 0, axis 0 0 1, limit lower=-1.9 upper=1.9 effort=0 velocity=0
- added joint 5392b5b20dc9647a: type revolute, parent 5392b5b2, child 0dc9647a, origin xyz=0.2 0 0 rpy=0 0 0, axis 0 0 1, limit lower=-1.9 upper=1.9 effort=0 velocity=0
- added joint 5392b5b29c2da2f4: type revolute, parent 5392b5b2, child 9c2da2f4, origin xyz=0 0.2 0 rpy=0 0 0, axis 0 0 1, limit lower=-1.9 upper=1.9 effort=0 velocity=0
- added joint 581c2250f49de8b1: type revolute, parent 581c2250, child f49de8b1, origin xyz=0 0.2 0 rpy=0 0 0, axis 0 0 1, limit lower=-1.9 upper=1.9 effort=0 velocity=0
- added joint 62d6a4e238092bac: type revolute, parent 62d6a4e2, child 38092bac, origin xyz=0 0.2 0 rpy=0 0 0, axis 0 0 1, limit lower=-1.9 upper=1.9 effort=0 velocity=0
- added joint 62d6a4e2b066414d: type revolute, parent 62d6a4e2, child b066414d, origin xyz=0 0.2 0 rpy=0 0 0, axis 0 0 1, limit lower=-1.9 upper=1.9 effort=0 velocity=0
- added joint 63bd3236d1ea9a80: type revolute, parent 63bd3236, child d1ea9a80, origin xyz=0 0.2 0 rpy=0 0 0, axis 0 0 1, limit lower=-1.9 upper=1.9 effort=0 velocity=0
- added joint 662e1da3b7a98a4a: type revolute, parent 662e1da3, child b7a98a4a, origin xyz=0 0.2 0 rpy=0 0 0, axis 0 0 1, limit lower=-1.9 upper=1.9 effort=0 velocity=0
- added joint 7187bc4c24b6d36c: type revolute, parent 7187bc4c, child 24b6d36c, origin xyz=0 0.2 0 rpy=0 0 0, axis 0 0 1, limit lower=-1.9 upper=1.9 effort=0 velocity=0
- added joint 734365891234c791: type revolute, parent 73436589, child 1234c791, origin xyz=0.2 0 0 rpy=0 0 0, axis 0 0 1, limit lower=-1.9 upper=1.9 effort=0 velocity=0
- added joint 73436589935073ed: type revolute, parent 73436589, child 935073ed, origin xyz=0 0.2 0 rpy=0 0 0, axis 0 0 1, limit lower=-1.9 upper=1.9 effort=0 velocity=0
- added joint 73436589d0ee7787: type revolute, parent 73436589, child d0ee7787, origin xyz=0.2 0 0 rpy=0 0 0, axis 0 0 1, limit lower=-1.9 upper=1.9 effort=0 velocity=0
- added joint 84c3bc2a63bd3236: type revolute, parent 84c3bc2a, child 63bd3236, origin xyz=0 0.2 0 rpy=0 0 0, axis 0 0 1, limit lower=-1.9 upper=1.9 effort=0 velocity=0
- added joint 9ec0e60062d6a4e2: type revolute, parent 9ec0e600, child 62d6a4e2, origin xyz=0 0.2 0 rpy=0 0 0, axis 0 0 1, limit lower=-1.9 upper=1.9 effort=0 velocity=0
- added joint a7ead54cc209a4f2: type revolute, parent a7ead54c, child c209a4f2, origin xyz=0 0.2 0 rpy=0 0 0, axis 0 0 1, limit lower=-1.9 upper=1.9 effort=0 velocity=0
- added joint a8351408f6724a8b: type revolute, parent a8351408, child f6724a8b, origin xyz=0 0.2 0 rpy=0 0 0, axis 0 0 1, limit lower=-1.9 upper=1.9 effort=0 velocity=0
- added joint adb2dd0fb3ea44e5: type revolute, parent adb2dd0f, child b3ea44e5, origin xyz=0 0.2 0 rpy=0 0 0, axis 0 0 1, limit lower=-1.9 upper=1.9 effort=0 velocity=0
- added joint b3ea44e543be07d9: type revolute, parent b3ea44e5, child 43be07d9, origin xyz=0 0.2 0 rpy=0 0 0, axis 0 0 1, limit lower=-1.9 upper=1.9 effort=0 velocity=0
- added joint b7a98a4adc94f799: type revolute, parent b7a98a4a, child dc94f799, origin xyz=0 0.2 0 rpy=0 0 0, axis 0 0 1, limit lower=-1.9 upper=1.9 effort=0 velocity=0
- added joint bc24cd03d779f3c3: type revolute, parent bc24cd03, child d779f3c3, origin xyz=0 0.2 0 rpy=0 0 0, axis 0 0 1, limit lower=-1.9 upper=1.9 effort=0 velocity=0
- added joint c209a4f268c0e889: type revolute, parent c209a4f2, child 68c0e889, origin xyz=0.2 0 0 rpy=0 0 0, axis 0 0 1, limit lower=-1.9 upper=1.9 effort=0 velocity=0
- added joint cd08ca7273436589: type revolute, parent cd08ca72, child 73436589, origin xyz=0 0.2 0 rpy=0 0 0, axis 0 0 1, limit lower=-1.9 upper=1.9 effort=0 velocity=0
- added joint d1ea9a80c0a43814: type revolute, parent d1ea9a80, child c0a43814, origin xyz=0 0.2 0 rpy=0 0 0, axis 0 0 1, limit lower=-1.9 upper=1.9 effort=0 velocity=0
- added joint d7336e025392b5b2: type revolute, parent d7336e02, child 5392b5b2, origin xyz=0 0.2 0 rpy=0 0 0, axis 0 0 1, limit lower=-1.9 upper=1.9 effort=0 velocity=0
- added joint d779f3c33a06f8cc: type revolute, parent d779f3c3, child 3a06f8cc, origin xyz=0 0.2 0 rpy=0 0 0, axis 0 0 1, limit lower=-1.9 upper=1.9 effort=0 velocity=0
- added joint dc94f79931c6b757: type revolute, parent dc94f799, child 31c6b757, origin xyz=0 0.2 0 rpy=0 0 0, axis 0 0 1, limit lower=-1.9 upper=1.9 effort=0 velocity=0
- added joint e400f108662e1da3: type revolute, parent e400f108, child 662e1da3, origin xyz=0 0.2 0 rpy=0 0 0, axis 0 0 1, limit lower=-1.9 upper=1.9 effort=0 velocity=0
- added joint f35b71d89ec0e600: type revolute, parent f35b71d8, child 9ec0e600, origin xyz=0.2 0 0 rpy=0 0 0, axis 0 0 1, limit lower=-1.9 upper=1.9 effort=0 velocity=0
- added joint f35b71d8ac6cf6e8: type revolute, parent f35b71d8, child ac6cf6e8, origin xyz=0 -0.2 0 rpy=0 0 0, axis 0 0 1, limit lower=-1.9 upper=1.9 effort=0 velocity=0
- added joint f35b71d8bcc4c2ba: type revolute, parent f35b71d8, child bcc4c2ba, origin xyz=0 0.2 0 rpy=0 0 0, axis 0 0 1, limit lower=-1.9 upper=1.9 effort=0 velocity=0
- added joint f49de8b1ff371f0e: type revolute, parent f49de8b1, child ff371f0e, origin xyz=0 0.2 0 rpy=0 0 0, axis 0 0 1, limit lower=-1.9 upper=1.9 effort=0 velocity=0
- added joint f8367eb9adb2dd0f: type revolute, parent f8367eb9, child adb2dd0f, origin xyz=0 0.2 0 rpy=0 0 0, axis 0 0 1, limit lower=-1.9 upper=1.9 effort=0 velocity=0
- added joint ff371f0e87d6d9a5: type revolute, parent ff371f0e, child 87d6d9a5, origin xyz=0 0.2 0 rpy=0 0 0, axis 0 0 1, limit lower=-1.9 upper=1.9 effort=0 velocity=0
