Commit message: Set up databases

File: parserTest.urdf (robot description, URDF)
Before this commit: robot paul, 604 links, 504 joints
Links:
- removed link 00015cb3
- removed link 0011a450
- removed link 008608bc
- removed link 00b83e39
- removed link 014e1755
- removed link 015259ad
- removed link 019d8163
- removed link 01e1af2e
- removed link 02425bfc
- removed link 037694ef
- removed link 0378e7de
- removed link 03b1ac4e
- removed link 04a10bd8
- removed link 04ad0b58
- removed link 05070f6c
- removed link 06c125a5
- removed link 07a55ca6
- removed link 085a6501
- removed link 086e4b9b
- removed link 088fb0f2
- removed link 08b31191
- removed link 0936e5a1
- removed link 093779da
- removed link 09d56e27
- removed link 0a015a04
- removed link 0a7904d5
- removed link 0a889ad3
- removed link 0b6f01c8
- removed link 0b728897
- removed link 0b83c886
- removed link 0be5c3b9
- removed link 0bf40198
- removed link 0bfa3c73
- removed link 0c634465
- removed link 0d51d491
- removed link 0d78c9ad
- removed link 0db19e7d
- removed link 0ddf995f
- removed link 0e4d2716
- removed link 0e8924b0
- removed link 0eaff118
- removed link 0ebaefdd
- removed link 0ec53256
- removed link 0f49b62c
- removed link 101e8254
- removed link 1243faaa
- removed link 137dc252
- removed link 1385a336
- removed link 13c84d04
- removed link 13e122f3
- removed link 142609e2
- removed link 14685b61
- removed link 146922f7
- removed link 14a3d1f7
- removed link 14ec2c48
- removed link 1530bf24
- removed link 15a730bb
- removed link 15d4ef5d
- removed link 16a8601e
- removed link 170e133a
- removed link 18501486
- removed link 189bc307
- removed link 18a776d7
- removed link 194bcc26
- removed link 197181a9
- removed link 19864c10
- removed link 1994f300
- removed link 1a0cd3b6
- removed link 1a2a4130
- removed link 1b057ba5
- removed link 1b07fb72
- removed link 1cae003d
- removed link 1d62cef1
- removed link 1df4485f
- removed link 1e28ceaa
- removed link 1e4c8cc6
- removed link 1fd8261c
- removed link 203415eb
- removed link 2090b5a6
- removed link 20a0efe2
- removed link 210ed15f
- removed link 216e20d7
- removed link 21d77b70
- removed link 22898709
- removed link 22f88d3e
- removed link 233ab126
- removed link 23549791
- removed link 2459e829
- removed link 24e14e44
- removed link 250f360a
- removed link 251ffd05
- removed link 25b4257b
- removed link 25bab453
- removed link 25f717b1
- removed link 27b3926f
- removed link 2902bfef
- removed link 299722db
- removed link 299d3cc7
- removed link 2a2f3ed0
- removed link 2a388459
- removed link 2a4bb69d
- removed link 2b889b5b
- removed link 2b9161ae
- removed link 2c6f3f23
- removed link 2ca880ba
- removed link 2cb10c65
- removed link 2cb95699
- removed link 30496a0e
- removed link 3106dcf7
- removed link 31e627fe
- removed link 32463a5f
- removed link 32bb24bb
- removed link 32d8ebf6
- removed link 337ded7b
- removed link 33f82c27
- removed link 3441d6cf
- removed link 348b2b12
- removed link 34cd27af
- removed link 34dcdba3
- removed link 35d62234
- removed link 3636ee1c
- removed link 366ecb9f
- removed link 36aea67f
- removed link 3781e380
- removed link 38054d20
- removed link 38843933
- removed link 39fa5478
- removed link 3a41d50e
- removed link 3b49fd95
- removed link 3b87f108
- removed link 3b8d01d0
- removed link 3bc83c16
- removed link 3bcb8eff
- removed link 3bf0f2f2
- removed link 3d0afdaa
- removed link 3d1dce2a
- removed link 3df47284
- removed link 3e532fe5
- removed link 3f9f6249
- removed link 407ded2c
- removed link 40b59602
- removed link 416bd1ac
- removed link 417ffafe
- removed link 41ac9302
- removed link 41efe348
- removed link 427ac5c2
- removed link 4371d3bc
- removed link 4386deb5
- removed link 439e1a4c
- removed link 43d3a479
- removed link 43e870c5
- removed link 447e035b
- removed link 456015a9
- removed link 457dd797
- removed link 45b87a4a
- removed link 45deed6b
- removed link 4604b865
- removed link 4657d2b0
- removed link 46f196c6
- removed link 475eceab
- removed link 486ef8d0
- removed link 48721f01
- removed link 48a80c0b
- removed link 49533b24
- removed link 4b38bed3
- removed link 4b4bd259
- removed link 4b6471cf
- removed link 4b774282
- removed link 4bded8c3
- removed link 4ccf9987
- removed link 4dc71744
- removed link 4de0fa7f
- removed link 4e0ef0b7
- removed link 4e177c55
- removed link 4e4d3ce4
- removed link 4e7d32d1
- removed link 4f215828
- removed link 4f24b422
- removed link 4f47bba2
- removed link 4fe3fcbe
- removed link 509da12d
- removed link 519101d2
- removed link 51b071bb
- removed link 5212a866
- removed link 5272d87b
- removed link 539666dc
- removed link 53988d8d
- removed link 53a3cb45
- removed link 547d4d41
- removed link 54c112a6
- removed link 552b4330
- removed link 55dc50c6
- removed link 5620c5e3
- removed link 5648b59d
- removed link 57322c24
- removed link 579a56db
- removed link 57f9293c
- removed link 581fc33f
- removed link 58236c56
- removed link 590cdb45
- removed link 5a20e818
- removed link 5b0db32c
- removed link 5c77e953
- removed link 5c8edee8
- removed link 5d88e372
- removed link 5de72288
- removed link 5e94bffa
- removed link 5fab1bc8
- removed link 600921b9
- removed link 6085af21
- removed link 60d9a0ae
- removed link 616a9524
- removed link 6218a30c
- removed link 62a86db2
- removed link 62e10326
- removed link 6320e2d7
- removed link 640a332a
- removed link 6455d29e
- removed link 66305e48
- removed link 666322c6
- removed link 66c9f657
- removed link 66f60948
- removed link 6705d8d7
- removed link 67418193
- removed link 67c91bbc
- removed link 67de4763
- removed link 688e1ed3
- removed link 68df4522
- removed link 68e0b55e
- removed link 699b46a8
- removed link 69bf82ae
- removed link 6a1ae27e
- removed link 6a330246
- removed link 6a376605
- removed link 6bbb0e5b
- removed link 6c3bd515
- removed link 6cf70fca
- removed link 6d05d7ed
- removed link 6d62a0f7
- removed link 6dcb537f
- removed link 6e1acfac
- removed link 6e430af5
- removed link 6e620f84
- removed link 7060e433
- removed link 70e6ab3f
- removed link 7135e237
- removed link 719550da
- removed link 71b827c2
- removed link 721b4592
- removed link 727c45ed
- removed link 72be3097
- removed link 72c632b0
- removed link 730a4c3b
- removed link 733603cd
- removed link 73d5bd3b
- removed link 73d7f899
- removed link 759470d7
- removed link 761cde78
- removed link 763f5528
- removed link 7667dd0f
- removed link 7783c096
- removed link 77c06bc2
- removed link 7802f6b7
- removed link 78043700
- removed link 786af20b
- removed link 78722a3f
- removed link 78f262f9
- removed link 795c2af7
- removed link 79a16551
- removed link 79f345d1
- removed link 7a1ba6a7
- removed link 7a1eb5ec
- removed link 7b63b80a
- removed link 7d0742bc
- removed link 7da5fb43
- removed link 7e1aa74d
- removed link 7e2df673
- removed link 7e8e29e9
- removed link 7f64b6f8
- removed link 802832fc
- removed link 802b9092
- removed link 808c7f73
- removed link 80a585df
- removed link 80fa11fd
- removed link 812291c6
- removed link 81fa810d
- removed link 82a7106d
- removed link 82e61cfe
- removed link 83a04738
- removed link 83e55ed7
- removed link 857c7e83
- removed link 85858fd4
- removed link 85bb8f4a
- removed link 86689f93
- removed link 873ed8bc
- removed link 8759c198
- removed link 8838baab
- removed link 88ca912d
- removed link 89398b32
- removed link 89f4f355
- removed link 8a38c34d
- removed link 8a468be4
- removed link 8a59159e
- removed link 8a8719a9
- removed link 8b10b4d6
- removed link 8b99c0d0
- removed link 8ba5a381
- removed link 8bbd9652
- removed link 8c689e6f
- removed link 8c79fac9
- removed link 8cd121df
- removed link 8dc53067
- removed link 8ddc08cf
- removed link 8dfb37d0
- removed link 8e205fbb
- removed link 8ed7eb10
- removed link 8f00d22f
- removed link 8fa6d780
- removed link 9052eeaa
- removed link 90b94be1
- removed link 90ecb3d0
- removed link 916fce5e
- removed link 91dab717
- removed link 9226a735
- removed link 9330c034
- removed link 93324e7e
- removed link 93505dbd
- removed link 94186ab7
- removed link 94837241
- removed link 94afe815
- removed link 94b1cbaa
- removed link 96ac8d73
- removed link 972395f8
- removed link 991473d5
- removed link 99218f05
- removed link 9981b866
- removed link 99b9a9d3
- removed link 9a148d83
- removed link 9a33a61c
- removed link 9a6fcec5
- removed link 9aaf7fc3
- removed link 9af595b0
- removed link 9be7a024
- removed link 9c00ce48
- removed link 9c1d3d5b
- removed link 9ca5a1e0
- removed link 9ca9036c
- removed link 9d6f6dd8
- removed link 9df4e580
- removed link 9e135dc0
- removed link 9eded1e1
- removed link 9eebdcc6
- removed link 9f1d5eb5
- removed link 9f6dbeb6
- removed link 9fdaaba2
- removed link a18411a2
- removed link a18848c7
- removed link a1f6ab94
- removed link a22c7b17
- removed link a25a01ab
- removed link a27bcf3a
- removed link a28210aa
- removed link a29982e3
- removed link a302fbb3
- removed link a3406f5b
- removed link a3642823
- removed link a4058378
- removed link a45a498a
- removed link a50c3483
- removed link a50f7b93
- removed link a5bdf230
- removed link a61e1ede
- removed link a662d3e8
- removed link a6a98966
- removed link a6f8ddc6
- removed link a773c23f
- removed link a7baf39b
- removed link a83d5d64
- removed link a851a28a
- removed link a8cddda4
- removed link a98cc63f
- removed link aa72a265
- removed link aa78faca
- removed link aac40c4a
- removed link ab28ce69
- removed link ab51ec5b
- removed link ab661395
- removed link ac46c034
- removed link acbe164b
- removed link acdb59c6
- removed link ade70698
- removed link aea66bff
- removed link aeca46d9
- removed link af73dc8f
- removed link afa04a35
- removed link afc59009
- removed link afca8d6b
- removed link b0014e0b
- removed link b053801c
- removed link b07d8056
- removed link b187a3cb
- removed link b1ee9bfb
- removed link b26cabbc
- removed link b2bc1327
- removed link b2e13549
- removed link b440e41a
- removed link b46ed861
- removed link b471ffd4
- removed link b4c0694f
- removed link b4dc6a39
- removed link b4eca285
- removed link b5e91429
- removed link b607a8de
- removed link b635f5b7
- removed link b68c6a52
- removed link b7440ecb
- removed link b7543097
- removed link b787e011
- removed link b81e7dec
- removed link b8e3256d
- removed link b9a5e207
- removed link b9acbc57
- removed link ba1629bc
- removed link baaabe7d
- removed link bb14e547
- removed link bbc343fe
- removed link bc35a7e1
- removed link bcc165b1
- removed link bd22322f
- removed link bdf9f766
- removed link be39dc23
- removed link be670b44
- removed link be9248ef
- removed link bf21514d
- removed link c019c13e
- removed link c01f81e3
- removed link c03e6cac
- removed link c04eb654
- removed link c058da49
- removed link c16cf5ab
- removed link c1afeae2
- removed link c1fac74e
- removed link c24aa29f
- removed link c27eacd7
- removed link c2f5deb9
- removed link c38c4f9a
- removed link c3f83dde
- removed link c50ee541
- removed link c565ff8c
- removed link c5b54c79
- removed link c5c01b29
- removed link c5d74136
- removed link c60d998b
- removed link c685bce6
- removed link c6a49571
- removed link c6af5bd5
- removed link c723de24
- removed link c87204e8
- removed link c986da7b
- removed link c98a6e7a
- removed link ca25c4bd
- removed link ca7deaae
- removed link cab5ddc8
- removed link cab9f232
- removed link cabba2a7
- removed link caf38871
- removed link cccc8176
- removed link cd45ca84
- removed link cd63c6b9
- removed link cd96b16f
- removed link ce954ce8
- removed link cf0694d9
- removed link cf44b8aa
- removed link cf5a4cb2
- removed link cfd15906
- removed link d09279e0
- removed link d14038ef
- removed link d1d56641
- removed link d1e2c9f2
- removed link d21fbf5b
- removed link d302d9ba
- removed link d32344e0
- removed link d360057c
- removed link d37757f5
- removed link d3cf6297
- removed link d3ddc32c
- removed link d47ea626
- removed link d47f6158
- removed link d4dee2d3
- removed link d615b8ee
- removed link d61f16bf
- removed link d7d57bd0
- removed link d80440f8
- removed link d873f9f6
- removed link d8eeecbf
- removed link d965bd46
- removed link d97a4ec9
- removed link d9c1a61e
- removed link da21e1f1
- removed link da306c13
- removed link dabee284
- removed link db1eaae0
- removed link db585d53
- removed link db6bc8b6
- removed link db8815e9
- removed link dc24032b
- removed link dca6bd00
- removed link ddeefc8e
- removed link def3ad80
- removed link df7d2736
- removed link dfd7264c
- removed link e00101b5
- removed link e0246017
- removed link e066e8b6
- removed link e18349fe
- removed link e1bcea4e
- removed link e33e9aca
- removed link e464cbb0
- removed link e4af22fb
- removed link e51bd23b
- removed link e5eaa835
- removed link e617e7a5
- removed link e6604a88
- removed link e672c85a
- removed link e6adb976
- removed link e6f39d45
- removed link e7134a11
- removed link e73507d5
- removed link e7392151
- removed link e7621dfb
- removed link e76aa3a7
- removed link e76ed36e
- removed link e7c93722
- removed link e7fc769e
- removed link e801fdb5
- removed link e837d9e0
- removed link e8c967ac
- removed link e8cfbfdf
- removed link e8d8bf6e
- removed link eabea45e
- removed link eac80c08
- removed link eb717ef3
- removed link eba816d8
- removed link eba825dd
- removed link ec36c0e7
- removed link ed67fc1c
- removed link ee2fa1dd
- removed link ee5850d1
- removed link efbf73dd
- removed link efd11c63
- removed link f0323b2e
- removed link f05c80ef
- removed link f061e90e
- removed link f07f3d6f
- removed link f07f47d3
- removed link f0f8c1e9
- removed link f175fbb6
- removed link f1835ef4
- removed link f1e11047
- removed link f269dee5
- removed link f28f6329
- removed link f2cb46ae
- removed link f31e1a70
- removed link f320fb51
- removed link f3434eaf
- removed link f3937aa4
- removed link f406e4c5
- removed link f4129050
- removed link f46d1502
- removed link f4e76d07
- removed link f50f8185
- removed link f58d8b54
- removed link f5b7e8ab
- removed link f5c5dffe
- removed link f67b2145
- removed link f699b24d
- removed link f6c8917f
- removed link f6cc143a
- removed link f7a02eea
- removed link f86cdbcc
- removed link f911f27e
- removed link f97c7901
- removed link f991876b
- removed link f9dfac25
- removed link fa27bd75
- removed link faaf65f2
- removed link fab1f2d0
- removed link fab44c8c
- removed link fb336f2d
- removed link fb403c97
- removed link fbce9f78
- removed link fc0a69f7
- removed link fc41d8b2
- removed link fc98f7da
- removed link fcae9f02
- removed link fce0fdbd
- removed link fd6707bf
- removed link fd83dfc3
- removed link fe119af1
- removed link fe4206f7
- removed link febe2f5b
- removed link ff2951fb
- removed link ff9da5ff
- removed link ffedd5ae
- added link 0ad44276, mass 1; collision box size=0.2 0.2 0.2; visual box size=0.2 0.2 0.2
- added link 0d01f08f, mass 1; collision box size=0.2 0.2 0.2; visual box size=0.2 0.2 0.2
- added link 0ff10355, mass 1; collision box size=0.2 0.2 0.2; visual box size=0.2 0.2 0.2
- added link 15cdb7e9, mass 1; collision box size=0.2 0.2 0.2; visual box size=0.2 0.2 0.2
- added link 2b03bbd1, mass 1; collision box size=0.2 0.2 0.2; visual box size=0.2 0.2 0.2
- added link 3d795317, mass 1; collision box size=0.2 0.2 0.2; visual box size=0.2 0.2 0.2
- added link 445de769, mass 1; collision box size=0.2 0.2 0.2; visual box size=0.2 0.2 0.2
- added link 52b3294b, mass 1; collision box size=0.2 0.2 0.2; visual box size=0.2 0.2 0.2
- added link 579f795f, mass 1; collision box size=0.2 0.2 0.2; visual box size=0.2 0.2 0.2
- added link 7b78bc8d, mass 1; collision box size=0.2 0.2 0.2; visual box size=0.2 0.2 0.2
- added link 89ee06c9, mass 1; collision box size=0.2 0.2 0.2; visual box size=0.2 0.2 0.2
- added link 94a11e2a, mass 1; collision box size=0.2 0.2 0.2; visual box size=0.2 0.2 0.2
- added link 9c54f725, mass 1; collision box size=0.2 0.2 0.2; visual box size=0.2 0.2 0.2
- added link 9d9e4a5f, mass 1; collision box size=0.2 0.2 0.2; visual box size=0.2 0.2 0.2
- added link aafcaa06, mass 1; collision box size=0.2 0.2 0.2; visual box size=0.2 0.2 0.2
- added link abb0d0e2, mass 1; collision box size=0.2 0.2 0.2; visual box size=0.2 0.2 0.2
- added link aea57d7d, mass 1; collision box size=0.2 0.2 0.2; visual box size=0.2 0.2 0.2
- added link b377d402, mass 1; collision box size=0.2 0.2 0.2; visual box size=0.2 0.2 0.2
- added link b41103dc, mass 1; collision box size=0.2 0.2 0.2; visual box size=0.2 0.2 0.2
- added link cd4a8334, mass 1; collision box size=0.2 0.2 0.2; visual box size=0.2 0.2 0.2
- added link d0c6494f, mass 1; collision box size=0.2 0.2 0.2; visual box size=0.2 0.2 0.2
- added link d775d82f, mass 1; collision box size=0.2 0.2 0.2; visual box size=0.2 0.2 0.2
Joints:
- removed joint 0011a450afca8d6b
- removed joint 014e1755a5bdf230
- removed joint 014e1755c60d998b
- removed joint 015259ad3781e380
- removed joint 015259adf0323b2e
- removed joint 019d8163df7d2736
- removed joint 01e1af2ef07f47d3
- removed joint 02425bfc1cae003d
- removed joint 02425bfc5e94bffa
- removed joint 037694efba1629bc
- removed joint 037694efff9da5ff
- removed joint 0378e7de58236c56
- removed joint 0378e7de6320e2d7
- removed joint 0378e7dedfd7264c
- removed joint 03b1ac4e552b4330
- removed joint 03b1ac4ed21fbf5b
- removed joint 04a10bd83a41d50e
- removed joint 05070f6cda306c13
- removed joint 06c125a50a7904d5
- removed joint 085a65013bc83c16
- removed joint 085a6501719550da
- removed joint 085a6501802b9092
- removed joint 085a65018a8719a9
- removed joint 085a65019a33a61c
- removed joint 086e4b9b9af595b0
- removed joint 088fb0f2f5c5dffe
- removed joint 08b311919a148d83
- removed joint 0936e5a141efe348
- removed joint 09d56e2778f262f9
- removed joint 0a015a040e4d2716
- removed joint 0a7904d5e76ed36e
- removed joint 0a889ad372be3097
- removed joint 0a889ad3795c2af7
- removed joint 0b6f01c82ca880ba
- removed joint 0b7288979df4e580
- removed joint 0b83c8864386deb5
- removed joint 0b83c88667418193
- removed joint 0b83c8869d6f6dd8
- removed joint 0b83c886c27eacd7
- removed joint 0be5c3b9a29982e3
- removed joint 0c63446513c84d04
- removed joint 0d51d491251ffd05
- removed joint 0d51d491b0014e0b
- removed joint 0d51d491e6adb976
- removed joint 0d78c9ad0936e5a1
- removed joint 0db19e7d2a388459
- removed joint 0ddf995fb4eca285
- removed joint 0e4d2716ff2951fb
- removed joint 0e8924b03f9f6249
- removed joint 0e8924b0547d4d41
- removed joint 0ebaefdd67c91bbc
- removed joint 0ec5325689f4f355
- removed joint 0f49b62c53988d8d
- removed joint 0f49b62cf699b24d
- removed joint 101e8254e00101b5
- removed joint 1243faaa68e0b55e
- removed joint 142609e2d360057c
- removed joint 14a3d1f7db585d53
- removed joint 14ec2c48b787e011
- removed joint 15a730bb4de0fa7f
- removed joint 15d4ef5d69bf82ae
- removed joint 170e133a9eded1e1
- removed joint 170e133aaac40c4a
- removed joint 185014866e620f84
- removed joint 18a776d76e1acfac
- removed joint 18a776d7efbf73dd
- removed joint 194bcc2605070f6c
- removed joint 197181a9539666dc
- removed joint 1994f300759470d7
- removed joint 1994f30080a585df
- removed joint 1994f3009fdaaba2
- removed joint 1a2a4130c5d74136
- removed joint 1b057ba5427ac5c2
- removed joint 1b057ba55b0db32c
- removed joint 1d62cef199218f05
- removed joint 1e28ceaa407ded2c
- removed joint 1e4c8cc606c125a5
- removed joint 216e20d7916fce5e
- removed joint 216e20d7f320fb51
- removed joint 22898709802832fc
- removed joint 22f88d3e6d05d7ed
- removed joint 2354979114a3d1f7
- removed joint 250f360a2c6f3f23
- removed joint 250f360acccc8176
- removed joint 25bab45362a86db2
- removed joint 25f717b1a45a498a
- removed joint 25f717b1cf5a4cb2
- removed joint 2902bfef8dfb37d0
- removed joint 2902bfefb26cabbc
- removed joint 299722db82a7106d
- removed joint 2a2f3ed07a1eb5ec
- removed joint 2a2f3ed08ddc08cf
- removed joint 2a388459640a332a
- removed joint 2a4bb69d3441d6cf
- removed joint 2b889b5b2cb95699
- removed joint 2b889b5b5c8edee8
- removed joint 2b889b5b9f1d5eb5
- removed joint 2cb10c65015259ad
- removed joint 30496a0ef3937aa4
- removed joint 31e627fe73d7f899
- removed joint 32463a5fab51ec5b
- removed joint 32bb24bb23549791
- removed joint 337ded7b41ac9302
- removed joint 337ded7bcf0694d9
- removed joint 33f82c2708b31191
- removed joint 33f82c27be9248ef
- removed joint 3441d6cf1a2a4130
- removed joint 3441d6cf7d0742bc
- removed joint 348b2b1204ad0b58
- removed joint 348b2b1221d77b70
- removed joint 348b2b12d4dee2d3
- removed joint 348b2b12ed67fc1c
- removed joint 34dcdba301e1af2e
- removed joint 3636ee1cbbc343fe
- removed joint 366ecb9fe8c967ac
- removed joint 38054d2094186ab7
- removed joint 38054d20e18349fe
- removed joint 39fa5478b607a8de
- removed joint 39fa5478dc24032b
- removed joint 3a41d50e14ec2c48
- removed joint 3b49fd95ab661395
- removed joint 3b8d01d02b889b5b
- removed joint 3bcb8eff27b3926f
- removed joint 3bf0f2f2bc35a7e1
- removed joint 3bf0f2f2e6f39d45
- removed joint 3d0afdaa7e2df673
- removed joint 3d1dce2ae51bd23b
- removed joint 407ded2c04a10bd8
- removed joint 417ffafeb5e91429
- removed joint 41efe3487da5fb43
- removed joint 427ac5c25de72288
- removed joint 4386deb5008608bc
- removed joint 4386deb535d62234
- removed joint 4386deb58a59159e
- removed joint 439e1a4c77c06bc2
- removed joint 43d3a479d47f6158
- removed joint 43e870c56a330246
- removed joint 43e870c5fb336f2d
- removed joint 456015a9337ded7b
- removed joint 45b87a4ae33e9aca
- removed joint 45deed6b96ac8d73
- removed joint 45deed6bf9dfac25
- removed joint 4657d2b070e6ab3f
- removed joint 4657d2b0e7392151
- removed joint 475eceabb053801c
- removed joint 475eceabd7d57bd0
- removed joint 48721f0185bb8f4a
- removed joint 48721f01a1f6ab94
- removed joint 48721f01fa27bd75
- removed joint 49533b244ccf9987
- removed joint 4b38bed351b071bb
- removed joint 4b6471cf1385a336
- removed joint 4b6471cf24e14e44
- removed joint 4bded8c338843933
- removed joint 4bded8c3f58d8b54
- removed joint 4ccf9987786af20b
- removed joint 4de0fa7f0c634465
- removed joint 4de0fa7fb2e13549
- removed joint 4e0ef0b7170e133a
- removed joint 4e177c55bcc165b1
- removed joint 4e4d3ce4f7a02eea
- removed joint 4e7d32d1fd6707bf
- removed joint 4f24b422146922f7
- removed joint 4f24b422f4e76d07
- removed joint 4fe3fcbe31e627fe
- removed joint 4fe3fcbe688e1ed3
- removed joint 519101d2b46ed861
- removed joint 51b071bbbe39dc23
- removed joint 5212a8668759c198
- removed joint 539666dcec36c0e7
- removed joint 53988d8d600921b9
- removed joint 53988d8d8bbd9652
- removed joint 53a3cb454604b865
- removed joint 54c112a61994f300
- removed joint 54c112a625b4257b
- removed joint 55dc50c60e8924b0
- removed joint 57322c24bb14e547
- removed joint 57f9293cafc59009
- removed joint 5a20e81834dcdba3
- removed joint 5c8edee80d51d491
- removed joint 5de722889ca5a1e0
- removed joint 5de72288b635f5b7
- removed joint 5e94bffab440e41a
- removed joint 5e94bffafebe2f5b
- removed joint 5fab1bc8873ed8bc
- removed joint 616a9524a6a98966
- removed joint 616a9524dabee284
- removed joint 6455d29eeba825dd
- removed joint 6455d29efcae9f02
- removed joint 666322c678722a3f
- removed joint 6705d8d785858fd4
- removed joint 6705d8d7e0246017
- removed joint 67de47630be5c3b9
- removed joint 68df45221b057ba5
- removed joint 68e0b55e67de4763
- removed joint 699b46a8b7440ecb
- removed joint 69bf82aeb68c6a52
- removed joint 6a376605a83d5d64
- removed joint 6c3bd515fab44c8c
- removed joint 6d05d7eda851a28a
- removed joint 6dcb537f2b9161ae
- removed joint 6dcb537f5212a866
- removed joint 6e1acface76aa3a7
- removed joint 6e430af5f67b2145
- removed joint 6e620f84c058da49
- removed joint 6e620f84eb717ef3
- removed joint 7060e433519101d2
- removed joint 7060e4338ba5a381
- removed joint 7135e237348b2b12
- removed joint 72be30977b63b80a
- removed joint 733603cd5620c5e3
- removed joint 73d5bd3bacbe164b
- removed joint 73d5bd3be4af22fb
- removed joint 73d7f8990a889ad3
- removed joint 73d7f8997e1aa74d
- removed joint 73d7f899efd11c63
- removed joint 761cde78d965bd46
- removed joint 7667dd0f7f64b6f8
- removed joint 7783c0961fd8261c
- removed joint 7783c096f86cdbcc
- removed joint 77c06bc2bdf9f766
- removed joint 77c06bc2cf44b8aa
- removed joint 7802f6b74e4d3ce4
- removed joint 78043700189bc307
- removed joint 786af20bb07d8056
- removed joint 78f262f91530bf24
- removed joint 78f262f96218a30c
- removed joint 79f345d148a80c0b
- removed joint 79f345d1c04eb654
- removed joint 7a1ba6a7f31e1a70
- removed joint 7b63b80acd96b16f
- removed joint 7da5fb439e135dc0
- removed joint 7da5fb43a4058378
- removed joint 7da5fb43dca6bd00
- removed joint 7e2df673acdb59c6
- removed joint 7e8e29e933f82c27
- removed joint 802832fcfc98f7da
- removed joint 802b9092439e1a4c
- removed joint 812291c68cd121df
- removed joint 812291c6aeca46d9
- removed joint 82a7106d972395f8
- removed joint 82e61cfeade70698
- removed joint 857c7e8313e122f3
- removed joint 857c7e8332d8ebf6
- removed joint 857c7e834b4bd259
- removed joint 857c7e839eebdcc6
- removed joint 873ed8bcf97c7901
- removed joint 89398b3214685b61
- removed joint 89398b324f215828
- removed joint 89f4f35583e55ed7
- removed joint 8a38c34d203415eb
- removed joint 8a38c34dd37757f5
- removed joint 8a38c34de5eaa835
- removed joint 8a59159ea302fbb3
- removed joint 8b10b4d622f88d3e
- removed joint 8b99c0d0142609e2
- removed joint 8c689e6ff406e4c5
- removed joint 8c689e6ffab1f2d0
- removed joint 8cd121df8e205fbb
- removed joint 8cd121df9a6fcec5
- removed joint 8dc530674f24b422
- removed joint 8ddc08cfa61e1ede
- removed joint 8ed7eb10faaf65f2
- removed joint 8f00d22ff0f8c1e9
- removed joint 8fa6d780581fc33f
- removed joint 8fa6d780a18411a2
- removed joint 8fa6d780cfd15906
- removed joint 9052eeaa5c77e953
- removed joint 9052eeaa6a1ae27e
- removed joint 9052eeaad3cf6297
- removed joint 90ecb3d0447e035b
- removed joint 90ecb3d05a20e818
- removed joint 9330c0349f6dbeb6
- removed joint 93324e7e8a38c34d
- removed joint 93505dbddb1eaae0
- removed joint 94186ab7d47ea626
- removed joint 9483724172c632b0
- removed joint 94837241763f5528
- removed joint 94837241f50f8185
- removed joint 94afe815a50f7b93
- removed joint 972395f8eabea45e
- removed joint 99218f054b774282
- removed joint 9981b8663b87f108
- removed joint 9981b8664371d3bc
- removed joint 99b9a9d3d61f16bf
- removed joint 99b9a9d3e617e7a5
- removed joint 9a6fcec5a8cddda4
- removed joint 9aaf7fc319864c10
- removed joint 9af595b0fc41d8b2
- removed joint 9af595b0fd83dfc3
- removed joint 9c00ce4879f345d1
- removed joint 9ca9036c6d62a0f7
- removed joint 9ca9036ccd63c6b9
- removed joint 9df4e580b471ffd4
- removed joint 9eebdcc64b38bed3
- removed joint 9eebdcc660d9a0ae
- removed joint 9eebdcc68a468be4
- removed joint 9eebdcc6ce954ce8
- removed joint 9f6dbeb6416bd1ac
- removed joint 9f6dbeb6e6604a88
- removed joint 9fdaaba2f269dee5
- removed joint a18411a28b10b4d6
- removed joint a22c7b1794837241
- removed joint a27bcf3acaf38871
- removed joint a28210aac5c01b29
- removed joint a302fbb3a98cc63f
- removed joint a3642823509da12d
- removed joint a50c3483f05c80ef
- removed joint a50f7b93616a9524
- removed joint a61e1ede299d3cc7
- removed joint a61e1ede6085af21
- removed joint a61e1edea7baf39b
- removed joint a61e1edef6c8917f
- removed joint a662d3e8a50c3483
- removed joint a6a98966b1ee9bfb
- removed joint a6f8ddc60bf40198
- removed joint a6f8ddc64657d2b0
- removed joint a851a28aa28210aa
- removed joint a8cddda4fbce9f78
- removed joint aa72a265666322c6
- removed joint ab28ce690a015a04
- removed joint ab51ec5b194bcc26
- removed joint acdb59c60ec53256
- removed joint acdb59c61a0cd3b6
- removed joint acdb59c6d302d9ba
- removed joint ade7069800b83e39
- removed joint ade7069848721f01
- removed joint aea66bff07a55ca6
- removed joint aea66bffd09279e0
- removed joint afc59009e7c93722
- removed joint afc59009ee2fa1dd
- removed joint afca8d6b037694ef
- removed joint b0014e0bdef3ad80
- removed joint b07d80569ca9036c
- removed joint b1ee9bfb3106dcf7
- removed joint b1ee9bfbc50ee541
- removed joint b1ee9bfbfe4206f7
- removed joint b26cabbc73d5bd3b
- removed joint b2bc13278dc53067
- removed joint b46ed86181fa810d
- removed joint b471ffd4093779da
- removed joint b471ffd489398b32
- removed joint b471ffd4e73507d5
- removed joint b4c0694f0b728897
- removed joint b4dc6a39d14038ef
- removed joint b4eca285216e20d7
- removed joint b5e91429f991876b
- removed joint b607a8de7667dd0f
- removed joint b607a8dec16cf5ab
- removed joint b635f5b7c1afeae2
- removed joint b68c6a52a3642823
- removed joint b7440ecbf1835ef4
- removed joint b787e011210ed15f
- removed joint b787e011c6af5bd5
- removed joint b9a5e20739fa5478
- removed joint baaabe7d1e28ceaa
- removed joint baaabe7db8e3256d
- removed joint bbc343fec38c4f9a
- removed joint bcc165b18c79fac9
- removed joint bd22322f43d3a479
- removed joint be39dc23590cdb45
- removed joint bf21514d54c112a6
- removed joint c01f81e3b9a5e207
- removed joint c01f81e3cabba2a7
- removed joint c03e6cac9330c034
- removed joint c03e6cacb187a3cb
- removed joint c1afeae293505dbd
- removed joint c1fac74e9c1d3d5b
- removed joint c2f5deb91df4485f
- removed joint c2f5deb99052eeaa
- removed joint c2f5deb9af73dc8f
- removed joint c38c4f9a1b07fb72
- removed joint c38c4f9a62e10326
- removed joint c38c4f9a94b1cbaa
- removed joint c38c4f9aaa72a265
- removed joint c3f83ddedb8815e9
- removed joint c565ff8c20a0efe2
- removed joint c565ff8cbd22322f
- removed joint c5b54c79086e4b9b
- removed joint c5d74136be670b44
- removed joint c685bce62a4bb69d
- removed joint c685bce64dc71744
- removed joint c87204e871b827c2
- removed joint c87204e8812291c6
- removed joint c98a6e7a6e430af5
- removed joint ca7deaae808c7f73
- removed joint cab5ddc85648b59d
- removed joint cab9f232727c45ed
- removed joint cab9f232a27bcf3a
- removed joint caf3887186689f93
- removed joint caf38871b4dc6a39
- removed joint cd45ca84475eceab
- removed joint cd63c6b988ca912d
- removed joint cf44b8aaaa78faca
- removed joint cf44b8aafc0a69f7
- removed joint cf5a4cb2b2bc1327
- removed joint cf5a4cb2c723de24
- removed joint d09279e0f28f6329
- removed joint d1d56641299722db
- removed joint d1e2c9f23636ee1c
- removed joint d32344e00db19e7d
- removed joint d32344e0ddeefc8e
- removed joint d3ddc32c4e0ef0b7
- removed joint d4dee2d31d62cef1
- removed joint d4dee2d35272d87b
- removed joint d615b8ee3df47284
- removed joint d615b8ee9981b866
- removed joint d7d57bd0c019c13e
- removed joint d80440f8019d8163
- removed joint d873f9f615a730bb
- removed joint d8eeecbf00015cb3
- removed joint d8eeecbf2902bfef
- removed joint d8eeecbfc6a49571
- removed joint d965bd466455d29e
- removed joint d97a4ec9014e1755
- removed joint d9c1a61ef3434eaf
- removed joint da306c136cf70fca
- removed joint db1eaae00bfa3c73
- removed joint db585d5345deed6b
- removed joint db585d5346f196c6
- removed joint db6bc8b66c3bd515
- removed joint db8815e902425bfc
- removed joint dca6bd005d88e372
- removed joint df7d27363bf0f2f2
- removed joint e00101b5457dd797
- removed joint e00101b578043700
- removed joint e024601716a8601e
- removed joint e0246017aea66bff
- removed joint e33e9acae8cfbfdf
- removed joint e4af22fb66c9f657
- removed joint e4af22fbe1bcea4e
- removed joint e51bd23bd3ddc32c
- removed joint e5eaa835088fb0f2
- removed joint e617e7a5a22c7b17
- removed joint e617e7a5f061e90e
- removed joint e6f39d4579a16551
- removed joint e7134a11c5b54c79
- removed joint e739215134cd27af
- removed joint e739215138054d20
- removed joint e7392151486ef8d0
- removed joint e7621dfb9226a735
- removed joint e7621dfb991473d5
- removed joint e7621dfbb7543097
- removed joint e76aa3a7e8d8bf6e
- removed joint e801fdb54b6471cf
- removed joint e837d9e07a1ba6a7
- removed joint e8c967aca662d3e8
- removed joint e8c967acda21e1f1
- removed joint e8cfbfdf57322c24
- removed joint eac80c08366ecb9f
- removed joint eac80c08f911f27e
- removed joint eb717ef38838baab
- removed joint eb717ef3b9acbc57
- removed joint eba816d8d873f9f6
- removed joint eba825dd53a3cb45
- removed joint eba825ddca25c4bd
- removed joint ec36c0e7721b4592
- removed joint f0323b2e66305e48
- removed joint f05c80efc24aa29f
- removed joint f07f3d6ff46d1502
- removed joint f0f8c1e90ddf995f
- removed joint f175fbb60378e7de
- removed joint f1835ef4f2cb46ae
- removed joint f269dee57802f6b7
- removed joint f320fb5183a04738
- removed joint f3434eaf03b1ac4e
- removed joint f3434eaf579a56db
- removed joint f3434eafee5850d1
- removed joint f3937aa490ecb3d0
- removed joint f406e4c5d615b8ee
- removed joint f412905066f60948
- removed joint f46d15027060e433
- removed joint f58d8b54e7fc769e
- removed joint f58d8b54fce0fdbd
- removed joint f5b7e8ab32463a5f
- removed joint f5c5dffe3bcb8eff
- removed joint f6c8917f90b94be1
- removed joint f6c8917fafa04a35
- removed joint f6c8917fb81e7dec
- removed joint f6c8917fca7deaae
- removed joint f6cc143a45b87a4a
- removed joint f86cdbcc101e8254
- removed joint f86cdbcca18848c7
- removed joint f991876b8c689e6f
- removed joint faaf65f222898709
- removed joint fab44c8cac46c034
- removed joint fab44c8cc986da7b
- removed joint fb403c97137dc252
- removed joint fb403c97233ab126
- removed joint fb403c9780fa11fd
- removed joint fb403c97a773c23f
- removed joint fb403c97cab5ddc8
- removed joint fbce9f78a25a01ab
- removed joint fc41d8b22090b5a6
- removed joint fc98f7da0eaff118
- removed joint fc98f7da2459e829
- removed joint fc98f7da4bded8c3
- removed joint fd6707bf3d1dce2a
- removed joint fe119af1cd45ca84
- removed joint febe2f5be801fdb5
- removed joint ff2951fb9be7a024
- removed joint ff2951fbf1e11047
- removed joint ff9da5ff6bbb0e5b
- removed joint ffedd5aed9c1a61e
- added joint 0ad4427615cdb7e9: type revolute, parent 0ad44276, child 15cdb7e9, origin xyz=0.2 0 0 rpy=0 0 0, axis 0 0 1, limit lower=-1.9 upper=1.9 effort=0 velocity=0
- added joint 0ad44276b377d402: type revolute, parent 0ad44276, child b377d402, origin xyz=0 0.2 0 rpy=0 0 0, axis 0 0 1, limit lower=-1.9 upper=1.9 effort=0 velocity=0
- added joint 0ad44276d775d82f: type revolute, parent 0ad44276, child d775d82f, origin xyz=0 0.2 0 rpy=0 0 0, axis 0 0 1, limit lower=-1.9 upper=1.9 effort=0 velocity=0
- added joint 0d01f08f52b3294b: type revolute, parent 0d01f08f, child 52b3294b, origin xyz=0 0.2 0 rpy=0 0 0, axis 0 0 1, limit lower=-1.9 upper=1.9 effort=0 velocity=0
- added joint 0ff10355b41103dc: type revolute, parent 0ff10355, child b41103dc, origin xyz=0 0.2 0 rpy=0 0 0, axis 0 0 1, limit lower=-1.9 upper=1.9 effort=0 velocity=0
- added joint 15cdb7e989ee06c9: type revolute, parent 15cdb7e9, child 89ee06c9, origin xyz=0 0.2 0 rpy=0 0 0, axis 0 0 1, limit lower=-1.9 upper=1.9 effort=0 velocity=0
- added joint 2b03bbd194a11e2a: type revolute, parent 2b03bbd1, child 94a11e2a, origin xyz=0 0.2 0 rpy=0 0 0, axis 0 0 1, limit lower=-1.9 upper=1.9 effort=0 velocity=0
- added joint 445de769aea57d7d: type revolute, parent 445de769, child aea57d7d, origin xyz=0 0.2 0 rpy=0 0 0, axis 0 0 1, limit lower=-1.9 upper=1.9 effort=0 velocity=0
- added joint 52b3294b579f795f: type revolute, parent 52b3294b, child 579f795f, origin xyz=0 0.2 0 rpy=0 0 0, axis 0 0 1, limit lower=-1.9 upper=1.9 effort=0 velocity=0
- added joint 579f795f445de769: type revolute, parent 579f795f, child 445de769, origin xyz=0 0.2 0 rpy=0 0 0, axis 0 0 1, limit lower=-1.9 upper=1.9 effort=0 velocity=0
- added joint 7b78bc8dd0c6494f: type revolute, parent 7b78bc8d, child d0c6494f, origin xyz=0 0.2 0 rpy=0 0 0, axis 0 0 1, limit lower=-1.9 upper=1.9 effort=0 velocity=0
- added joint 89ee06c93d795317: type revolute, parent 89ee06c9, child 3d795317, origin xyz=0 0.2 0 rpy=0 0 0, axis 0 0 1, limit lower=-1.9 upper=1.9 effort=0 velocity=0
- added joint 89ee06c9abb0d0e2: type revolute, parent 89ee06c9, child abb0d0e2, origin xyz=0 0.2 0 rpy=0 0 0, axis 0 0 1, limit lower=-1.9 upper=1.9 effort=0 velocity=0
- added joint 89ee06c9cd4a8334: type revolute, parent 89ee06c9, child cd4a8334, origin xyz=0.2 0 0 rpy=0 0 0, axis 0 0 1, limit lower=-1.9 upper=1.9 effort=0 velocity=0
- added joint 9d9e4a5f7b78bc8d: type revolute, parent 9d9e4a5f, child 7b78bc8d, origin xyz=0 0.2 0 rpy=0 0 0, axis 0 0 1, limit lower=-1.9 upper=1.9 effort=0 velocity=0
- added joint aafcaa060ff10355: type revolute, parent aafcaa06, child 0ff10355, origin xyz=0 0.2 0 rpy=0 0 0, axis 0 0 1, limit lower=-1.9 upper=1.9 effort=0 velocity=0
- added joint abb0d0e22b03bbd1: type revolute, parent abb0d0e2, child 2b03bbd1, origin xyz=0 0.2 0 rpy=0 0 0, axis 0 0 1, limit lower=-1.9 upper=1.9 effort=0 velocity=0
- added joint b41103dc0d01f08f: type revolute, parent b41103dc, child 0d01f08f, origin xyz=0 0.2 0 rpy=0 0 0, axis 0 0 1, limit lower=-1.9 upper=1.9 effort=0 velocity=0
- added joint d0c6494f9c54f725: type revolute, parent d0c6494f, child 9c54f725, origin xyz=0 0.2 0 rpy=0 0 0, axis 0 0 1, limit lower=-1.9 upper=1.9 effort=0 velocity=0
- added joint d0c6494faafcaa06: type revolute, parent d0c6494f, child aafcaa06, origin xyz=0.2 0 0 rpy=0 0 0, axis 0 0 1, limit lower=-1.9 upper=1.9 effort=0 velocity=0
