Commit message: Separated evaluation into independent python file

File: parserTest.urdf (robot description, URDF)
Before this commit: robot paul, 22 links, 20 joints
Links:
- removed link 0ad44276
- removed link 0d01f08f
- removed link 0ff10355
- removed link 15cdb7e9
- removed link 2b03bbd1
- removed link 3d795317
- removed link 445de769
- removed link 52b3294b
- removed link 579f795f
- removed link 7b78bc8d
- removed link 89ee06c9
- removed link 94a11e2a
- removed link 9c54f725
- removed link 9d9e4a5f
- removed link aafcaa06
- removed link abb0d0e2
- removed link aea57d7d
- removed link b377d402
- removed link b41103dc
- removed link cd4a8334
- removed link d0c6494f
- removed link d775d82f
- added link 250b9131, mass 1; collision box size=0.2 0.2 0.2; visual box size=0.2 0.2 0.2
- added link 2af714b5, mass 1; collision box size=0.2 0.2 0.2; visual box size=0.2 0.2 0.2
- added link 3cb68742, mass 1; collision box size=0.2 0.2 0.2; visual box size=0.2 0.2 0.2
- added link 3cb9098e, mass 1; collision box size=0.2 0.2 0.2; visual box size=0.2 0.2 0.2
- added link bc2255c6, mass 1; collision box size=0.2 0.2 0.2; visual box size=0.2 0.2 0.2
- added link da68b957, mass 1; collision box size=0.2 0.2 0.2; visual box size=0.2 0.2 0.2
Joints:
- removed joint 0ad4427615cdb7e9
- removed joint 0ad44276b377d402
- removed joint 0ad44276d775d82f
- removed joint 0d01f08f52b3294b
- removed joint 0ff10355b41103dc
- removed joint 15cdb7e989ee06c9
- removed joint 2b03bbd194a11e2a
- removed joint 445de769aea57d7d
- removed joint 52b3294b579f795f
- removed joint 579f795f445de769
- removed joint 7b78bc8dd0c6494f
- removed joint 89ee06c93d795317
- removed joint 89ee06c9abb0d0e2
- removed joint 89ee06c9cd4a8334
- removed joint 9d9e4a5f7b78bc8d
- removed joint aafcaa060ff10355
- removed joint abb0d0e22b03bbd1
- removed joint b41103dc0d01f08f
- removed joint d0c6494f9c54f725
- removed joint d0c6494faafcaa06
- added joint 3cb9098e2af714b5: type revolute, parent 3cb9098e, child 2af714b5, origin xyz=0 0.2 0 rpy=0 0 0, axis 0 0 1, limit lower=-1.9 upper=1.9 effort=0 velocity=0
- added joint bc2255c6250b9131: type revolute, parent bc2255c6, child 250b9131, origin xyz=0 0.2 0 rpy=0 0 0, axis 0 0 1, limit lower=-1.9 upper=1.9 effort=0 velocity=0
- added joint bc2255c63cb68742: type revolute, parent bc2255c6, child 3cb68742, origin xyz=0 0.2 0 rpy=0 0 0, axis 0 0 1, limit lower=-1.9 upper=1.9 effort=0 velocity=0
- added joint bc2255c63cb9098e: type revolute, parent bc2255c6, child 3cb9098e, origin xyz=0 -0.2 0 rpy=0 0 0, axis 0 0 1, limit lower=-1.9 upper=1.9 effort=0 velocity=0
- added joint da68b957bc2255c6: type revolute, parent da68b957, child bc2255c6, origin xyz=0 0.2 0 rpy=0 0 0, axis 0 0 1, limit lower=-1.9 upper=1.9 effort=0 velocity=0

Commit message: Various upgrades and fixes

File: parserTest.urdf (robot description, URDF)
Before this commit: robot paul, 6 links, 5 joints
Links:
- removed link 250b9131
- removed link 2af714b5
- removed link 3cb68742
- removed link 3cb9098e
- removed link bc2255c6
- removed link da68b957
- added link 6fc645df, mass 1; collision box size=0.2 0.2 0.2; visual box size=0.2 0.2 0.2
- added link 7d984038, mass 1; collision box size=0.2 0.2 0.2; visual box size=0.2 0.2 0.2
- added link 981639e8, mass 1; collision box size=0.2 0.2 0.2; visual box size=0.2 0.2 0.2
- added link eb3d5164, mass 1; collision box size=0.2 0.2 0.2; visual box size=0.2 0.2 0.2
- added link f764cc10, mass 1; collision box size=0.2 0.2 0.2; visual box size=0.2 0.2 0.2
Joints:
- removed joint 3cb9098e2af714b5
- removed joint bc2255c6250b9131
- removed joint bc2255c63cb68742
- removed joint bc2255c63cb9098e
- removed joint da68b957bc2255c6
- added joint 7d984038f764cc10: type revolute, parent 7d984038, child f764cc10, origin xyz=0 0.2 0 rpy=0 0 0, axis 0 0 1, limit lower=-1.9 upper=1.9 effort=0 velocity=0
- added joint 981639e86fc645df: type revolute, parent 981639e8, child 6fc645df, origin xyz=0 0.2 0 rpy=0 0 0, axis 0 0 1, limit lower=-1.9 upper=1.9 effort=0 velocity=0
- added joint eb3d5164981639e8: type revolute, parent eb3d5164, child 981639e8, origin xyz=0 0.2 0 rpy=0 0 0, axis 0 0 1, limit lower=-1.9 upper=1.9 effort=0 velocity=0
- added joint f764cc10eb3d5164: type revolute, parent f764cc10, child eb3d5164, origin xyz=0 0.2 0 rpy=0 0 0, axis 0 0 1, limit lower=-1.9 upper=1.9 effort=0 velocity=0
