Commit message: Added parsing for parameters

File: robot.urdf (robot description, URDF)
Before this commit: robot paul, 2 links, 1 joints
Links:
- removed link 331e4408
- removed link fa1cb030
- added link 905f28be, mass 1; collision box size=0.2 0.2 0.2; visual box size=0.2 0.2 0.2
- added link e505a4d5, mass 1; collision box size=0.2 0.2 0.2; visual box size=0.2 0.2 0.2
Joints:
- removed joint 331e4408fa1cb030
- added joint e505a4d5905f28be: type revolute, parent e505a4d5, child 905f28be, origin xyz=-0.2 0 0 rpy=0 0 0, axis 0 0 1, limit lower=-1.9 upper=1.9 effort=0 velocity=0

Commit message: Fixed index out of range error for parameters near end of string

File: robot.urdf (robot description, URDF)
Before this commit: robot paul, 2 links, 1 joints
Links:
- removed link 905f28be
- removed link e505a4d5
- added link 396733bf, mass 1; collision box size=0.2 0.2 0.2; visual box size=0.2 0.2 0.2
- added link 4059a773, mass 1; collision box size=0.2 0.2 0.2; visual box size=0.2 0.2 0.2
- added link 6a81c18c, mass 1; collision box size=0.2 0.2 0.2; visual box size=0.2 0.2 0.2
- added link 8f912c0d, mass 1; collision box size=0.2 0.2 0.2; visual box size=0.2 0.2 0.2
Joints:
- removed joint e505a4d5905f28be
- added joint 396733bf4059a773: type revolute, parent 396733bf, child 4059a773, origin xyz=-0.2 0 0 rpy=0 0 0, axis 0 0 1, limit lower=-1.9 upper=1.9 effort=0 velocity=0
- added joint 396733bf8f912c0d: type revolute, parent 396733bf, child 8f912c0d, origin xyz=-0.2 0 0 rpy=0 0 0, axis 0 0 1, limit lower=-1.9 upper=1.9 effort=0 velocity=0
- added joint 8f912c0d6a81c18c: type revolute, parent 8f912c0d, child 6a81c18c, origin xyz=-0.2 0 0 rpy=0 0 0, axis 0 0 1, limit lower=-1.9 upper=1.9 effort=0 velocity=0

Commit message: Added support for parameters in parser.py

File: robot.urdf (robot description, URDF)
Before this commit: robot paul, 4 links, 3 joints
Links:
- removed link 396733bf
- removed link 4059a773
- removed link 6a81c18c
- removed link 8f912c0d
- added link 0e4e64ca, mass 3.0; collision box size=0.4 0.4 0.4; visual box size=0.4 0.4 0.4
- added link 66880f38, mass 1; collision box size=0.2 0.4 0.2; visual box size=0.2 0.4 0.2
- added link 7709b61b, mass 1; collision box size=0.4 0.2 0.2; visual box size=0.4 0.2 0.2
- added link abad6ce3, mass 1; collision box size=0.2 0.2 0.2; visual box size=0.2 0.2 0.2
Joints:
- removed joint 396733bf4059a773
- removed joint 396733bf8f912c0d
- removed joint 8f912c0d6a81c18c
- added joint 7709b61b66880f38: type revolute, parent 7709b61b, child 66880f38, origin xyz=0.0 0.0 -0.2 rpy=0 0 0, axis 1 0 0, limit lower=6.0 upper=5.0 effort=3.0 velocity=4.0
- added joint 7709b61babad6ce3: type revolute, parent 7709b61b, child abad6ce3, origin xyz=0.0 0.0 -0.2 rpy=0 0 0, axis 1 0 0, limit lower=-1.9 upper=1.9 effort=0 velocity=0
- added joint abad6ce30e4e64ca: type revolute, parent abad6ce3, child 0e4e64ca, origin xyz=-0.4 0.0 0.0 rpy=0 0 0, axis 0 1 0, limit lower=-1.9 upper=1.9 effort=0 velocity=0

Commit message: Still fixing mutations to work with parameters

File: robot.urdf (robot description, URDF)
Before this commit: robot paul, 4 links, 3 joints
Links:
- removed link 0e4e64ca
- removed link 66880f38
- removed link 7709b61b
- removed link abad6ce3
- added link 1b3c5158, mass 1; collision box size=1.2 0.64 0.2; visual box size=1.2 0.64 0.2
- added link 67b3bdd6, mass 1; collision box size=0.2 0.2 0.2; visual box size=0.2 0.2 0.2
- added link 8bf16970, mass 1; collision box size=0.02 0.0 0.2; visual box size=0.02 0.0 0.2
- added link a9a6fc60, mass 1; collision box size=0.2 0.2 0.2; visual box size=0.2 0.2 0.2
Joints:
- removed joint 7709b61b66880f38
- removed joint 7709b61babad6ce3
- removed joint abad6ce30e4e64ca
- added joint 1b3c51588bf16970: type revolute, parent 1b3c5158, child 8bf16970, origin xyz=0.0 0.0 -0.2 rpy=0 0 0, axis 0 1 0, limit lower=-1.9 upper=1.9 effort=0 velocity=0
- added joint 8bf16970a9a6fc60: type revolute, parent 8bf16970, child a9a6fc60, origin xyz=0.0 0.2 0.0 rpy=0 0 0, axis 0 0 1, limit lower=-1.9 upper=1.9 effort=0 velocity=0
- added joint a9a6fc6067b3bdd6: type revolute, parent a9a6fc60, child 67b3bdd6, origin xyz=0.0 0.2 0.0 rpy=0 0 0, axis 0 0 1, limit lower=-1.9 upper=1.9 effort=0 velocity=0

Commit message: Added commas to mutator to move cubes around

File: robot.urdf (robot description, URDF)
Before this commit: robot paul, 4 links, 3 joints
Links:
- removed link 1b3c5158
- removed link 67b3bdd6
- removed link 8bf16970
- removed link a9a6fc60
- added link 0443cef8, mass 0.587377537087; collision box size=0.0132225166836 0.0409653215416 0.0529219438702; visual box size=0.0132225166836 0.0409653215416 0.0529219438702
- added link 05fb6450, mass 0.773851986496; collision box size=0.100104259793 0.160221870822 0.0277337756608; visual box size=0.100104259793 0.160221870822 0.0277337756608
- added link 0b5a6eef, mass 0.17795049276; collision box size=0.0808027819192 0.227467787174 0.131840645988; visual box size=0.0808027819192 0.227467787174 0.131840645988
- added link 0cdc028b, mass 1; collision box size=0.0843382441056 0.0167173569684 0.2; visual box size=0.0843382441056 0.0167173569684 0.2
- added link 0f457723, mass 0.0562839946932; collision box size=0.232578626892 0.0340881376466 0.0486208371476; visual box size=0.232578626892 0.0340881376466 0.0486208371476
- added link 105cdbe8, mass 0.147974814275; collision box size=0.199247555533 0.236723511144 0.089660214895; visual box size=0.199247555533 0.236723511144 0.089660214895
- added link 14945161, mass 0.0725935453546; collision box size=0.0610886104192 0.00027782406243 0.227622919786; visual box size=0.0610886104192 0.00027782406243 0.227622919786
- added link 18b29c49, mass 0.594868004824; collision box size=0.0707930132382 0.246813578586 0.48747369748; visual box size=0.0707930132382 0.246813578586 0.48747369748
- added link 275c27f4, mass 0.341980497439; collision box size=0.128272554227 0.195171391337 0.151876556298; visual box size=0.128272554227 0.195171391337 0.151876556298
- added link 30fc0f2e, mass 1.34691255385; collision box size=0.033952604541 0.0156937658866 0.0510297654906; visual box size=0.033952604541 0.0156937658866 0.0510297654906
- added link 3156b1b7, mass 0.316442532757; collision box size=0.0679387894876 0.00957289119122 0.020176916447; visual box size=0.0679387894876 0.00957289119122 0.020176916447
- added link 3691be7d, mass 0.0868762881569; collision box size=0.111908339714 0.00513391865028 0.0450365789612; visual box size=0.111908339714 0.00513391865028 0.0450365789612
- added link 377fa558, mass 0.438689538383; collision box size=0.161215684376 0.0563476789502 0.00550104180834; visual box size=0.161215684376 0.0563476789502 0.00550104180834
- added link 3da6150c, mass 0.0650655309281; collision box size=0.0108870534431 0.0444796676004 0.145823653908; visual box size=0.0108870534431 0.0444796676004 0.145823653908
- added link 413041c7, mass 0.376307739183; collision box size=0.138968980934 0.0184764451506 0.056534615929; visual box size=0.138968980934 0.0184764451506 0.056534615929
- added link 4b7a5ff1, mass 0.0245540538144; collision box size=0.143559181786 0.0469090906098 0.24862996467; visual box size=0.143559181786 0.0469090906098 0.24862996467
- added link 591f5e18, mass 1; collision box size=0.131795017515 0.0212940119294 0.2; visual box size=0.131795017515 0.0212940119294 0.2
- added link 64c6f495, mass 0.215708115042; collision box size=0.45040473831 0.067132646337 0.0282919119518; visual box size=0.45040473831 0.067132646337 0.0282919119518
- added link 6842db81, mass 0.0347608842593; collision box size=1.24897414772 3.0449518764 3.37554395198; visual box size=1.24897414772 3.0449518764 3.37554395198
- added link 6ec480c8, mass 0.0599475888866; collision box size=0.0327007552234 0.296890064168 0.42189709814; visual box size=0.0327007552234 0.296890064168 0.42189709814
- added link 70a813a7, mass 1.03861954971; collision box size=0.0977121751532 0.0910591573796 0.0436593132692; visual box size=0.0977121751532 0.0910591573796 0.0436593132692
- added link 726e66ea, mass 0.670081779255; collision box size=0.0695114151006 0.110189683494 0.0154031405075; visual box size=0.0695114151006 0.110189683494 0.0154031405075
- added link 7890965f, mass 0.647623665562; collision box size=0.180373033082 0.10029180219 0.048116750126; visual box size=0.180373033082 0.10029180219 0.048116750126
- added link 7d2f91e4, mass 0.424167385001; collision box size=0.110378961481 0.0227442211358 0.170972890682; visual box size=0.110378961481 0.0227442211358 0.170972890682
- added link 83cccbd2, mass 0.996296461608; collision box size=0.0652540005542 0.107914655121 0.0258191701778; visual box size=0.0652540005542 0.107914655121 0.0258191701778
- added link 85decfd8, mass 0.506951091618; collision box size=0.0875968007704 0.0582290253912 0.125876742615; visual box size=0.0875968007704 0.0582290253912 0.125876742615
- added link 87d7940f, mass 0.471939396325; collision box size=0.0361416689892 0.0080074759284 0.111973493679; visual box size=0.0361416689892 0.0080074759284 0.111973493679
- added link 954daca0, mass 0.603282360309; collision box size=0.0265839089966 0.0677195858122 0.106725024906; visual box size=0.0265839089966 0.0677195858122 0.106725024906
- added link 982855a3, mass 0.303939301494; collision box size=0.13318379243 0.115377989296 0.188340843347; visual box size=0.13318379243 0.115377989296 0.188340843347
- added link 9b5bd92e, mass 0.583002862284; collision box size=0.0724202115472 0.0138951874763 0.0271435728634; visual box size=0.0724202115472 0.0138951874763 0.0271435728634
- added link 9cdb5009, mass 0.629287541202; collision box size=0.0480505025842 0.113004653739 0.161601279303; visual box size=0.0480505025842 0.113004653739 0.161601279303
- added link b5190963, mass 0.263191333129; collision box size=0.0501145990306 0.00454454445846 0.039425262923; visual box size=0.0501145990306 0.00454454445846 0.039425262923
- added link bb90fee0, mass 1; collision box size=0.2 0.2 0.2; visual box size=0.2 0.2 0.2
- added link c9507b8b, mass 0.111455865671; collision box size=0.0462533670282 0.0629544528298 0.0436530380084; visual box size=0.0462533670282 0.0629544528298 0.0436530380084
- added link d63c789b, mass 0.5931795356; collision box size=0.373904167994 0.000351354843484 0.0150291142307; visual box size=0.373904167994 0.000351354843484 0.0150291142307
- added link d78aac32, mass 0.302100867337; collision box size=0.16721342478 0.072733274844 0.0716992098832; visual box size=0.16721342478 0.072733274844 0.0716992098832
- added link e68ff6a4, mass 0.205619450237; collision box size=0.181134077942 0.106878170724 0.0349744380616; visual box size=0.181134077942 0.106878170724 0.0349744380616
- added link e8e5e8db, mass 0.228889692784; collision box size=0.495158420822 0.0764411391882 0.00885682867066; visual box size=0.495158420822 0.0764411391882 0.00885682867066
- added link ea98e739, mass 0.162360917893; collision box size=0.0741834445328 0.0549607904578 0.00177249207438; visual box size=0.0741834445328 0.0549607904578 0.00177249207438
- added link f3d7be28, mass 0.0840733723647; collision box size=0.0188345583162 0.0136163199279 0.158944847299; visual box size=0.0188345583162 0.0136163199279 0.158944847299
Joints:
- removed joint 1b3c51588bf16970
- removed joint 8bf16970a9a6fc60
- removed joint a9a6fc6067b3bdd6
- added joint 0443cef8591f5e18: type revolute, parent 0443cef8, child 591f5e18, origin xyz=-0.131795017515 0.0 0.0 rpy=0 0 0, axis 0 0 1, limit lower=-1.9 upper=1.9 effort=0.137300350857 velocity=0
- added joint 05fb645087d7940f: type revolute, parent 05fb6450, child 87d7940f, origin xyz=0.0 -0.0080074759284 0.0 rpy=0 0 0, axis 0 0 1, limit lower=-1.9 upper=0.118858956421 effort=0.362596929965 velocity=1.05859227301
- added joint 0b5a6eefea98e739: type revolute, parent 0b5a6eef, child ea98e739, origin xyz=0.0 0.0 0.00177249207438 rpy=0 0 0, axis 0 0 1, limit lower=-1.9 upper=0.812217877935 effort=0.155820395792 velocity=1.90733384287
- added joint 0cdc028bbb90fee0: type revolute, parent 0cdc028b, child bb90fee0, origin xyz=0.0 0.2 0.0 rpy=0 0 0, axis 0 0 1, limit lower=-1.9 upper=1.9 effort=0 velocity=0
- added joint 0f4577236842db81: type revolute, parent 0f457723, child 6842db81, origin xyz=0.0 0.0 3.37554395198 rpy=0 0 0, axis 0 0 1, limit lower=-1.9 upper=0.0612437944803 effort=0.341324818291 velocity=0.282177734903
- added joint 105cdbe89cdb5009: type revolute, parent 105cdbe8, child 9cdb5009, origin xyz=-0.0480505025842 0.0 0.0 rpy=0 0 0, axis 0 0 1, limit lower=-1.9 upper=0.732582262505 effort=0.853951852164 velocity=0.646667427174
- added joint 14945161377fa558: type revolute, parent 14945161, child 377fa558, origin xyz=0.0 0.0 0.00550104180834 rpy=0 0 0, axis 0 1 0, limit lower=-1.9 upper=0.087020882853 effort=0.201760570192 velocity=0.208178333362
- added joint 18b29c49f3d7be28: type revolute, parent 18b29c49, child f3d7be28, origin xyz=-0.0188345583162 0.0 0.0 rpy=0 0 0, axis 0 0 1, limit lower=-1.9 upper=0.860712528875 effort=0.0433088652767 velocity=1.8348265774
- added joint 275c27f4d78aac32: type revolute, parent 275c27f4, child d78aac32, origin xyz=0.0 -0.072733274844 0.0 rpy=0 0 0, axis 0 0 1, limit lower=-1.9 upper=0.385846507638 effort=0.0503900214603 velocity=0.430679895929
- added joint 30fc0f2e3156b1b7: type revolute, parent 30fc0f2e, child 3156b1b7, origin xyz=0.0 0.00957289119122 0.0 rpy=0 0 0, axis 0 0 1, limit lower=-1.9 upper=0.136287542501 effort=0.542107316538 velocity=0.383825736981
- added joint 3156b1b718b29c49: type revolute, parent 3156b1b7, child 18b29c49, origin xyz=0.0 0.0 -0.48747369748 rpy=0 0 0, axis 0 0 1, limit lower=-1.9 upper=0.0454098009483 effort=0.0261534036422 velocity=0.258218931186
- added joint 3691be7d30fc0f2e: type revolute, parent 3691be7d, child 30fc0f2e, origin xyz=0.0 -0.0156937658866 0.0 rpy=0 0 0, axis 0 0 1, limit lower=-1.9 upper=0.582318646095 effort=0.241636866455 velocity=0.11998356245
- added joint 377fa5584b7a5ff1: type revolute, parent 377fa558, child 4b7a5ff1, origin xyz=0.0 0.0 -0.24862996467 rpy=0 0 0, axis 0 0 1, limit lower=-1.9 upper=1.19717226534 effort=0.438887762208 velocity=0.82305196682
- added joint 3da6150c70a813a7: type revolute, parent 3da6150c, child 70a813a7, origin xyz=0.0977121751532 0.0 0.0 rpy=0 0 0, axis 0 0 1, limit lower=-1.9 upper=0.0819521360715 effort=0.142466965312 velocity=0.08895214737
- added joint 413041c7e68ff6a4: type revolute, parent 413041c7, child e68ff6a4, origin xyz=0.0 0.106878170724 0.0 rpy=0 0 0, axis 0 0 1, limit lower=-1.9 upper=0.654849995196 effort=0.0770955344402 velocity=0.00323336652077
- added joint 4b7a5ff10b5a6eef: type revolute, parent 4b7a5ff1, child 0b5a6eef, origin xyz=0.0 -0.227467787174 0.0 rpy=0 0 0, axis 0 0 1, limit lower=-1.9 upper=0.43609175347 effort=0.350386261313 velocity=0.713738375051
- added joint 591f5e180cdc028b: type revolute, parent 591f5e18, child 0cdc028b, origin xyz=0.0 0.0 0.2 rpy=0 0 0, axis 0 0 1, limit lower=-1.9 upper=1.9 effort=0.963560720648 velocity=0
- added joint 64c6f495275c27f4: type revolute, parent 64c6f495, child 275c27f4, origin xyz=0.0 0.0 -0.151876556298 rpy=0 0 0, axis 0 0 1, limit lower=-1.9 upper=0.0760317740144 effort=0.0757735697141 velocity=0.520221925372
- added joint 6842db81c9507b8b: type revolute, parent 6842db81, child c9507b8b, origin xyz=-0.0462533670282 0.0 0.0 rpy=0 0 0, axis 0 0 1, limit lower=-1.9 upper=0.505516101845 effort=0.12045645513 velocity=0.246351297771
- added joint 6ec480c8d63c789b: type revolute, parent 6ec480c8, child d63c789b, origin xyz=0.0 -0.000351354843484 0.0 rpy=0 0 0, axis 0 1 0, limit lower=-1.9 upper=0.263953655824 effort=0.692193661504 velocity=0.416836502422
- added joint 70a813a77890965f: type revolute, parent 70a813a7, child 7890965f, origin xyz=0.180373033082 0.0 0.0 rpy=0 0 0, axis 0 0 1, limit lower=-1.9 upper=0.452427880046 effort=0.209822824673 velocity=0.319225240367
- added joint 726e66ea0443cef8: type revolute, parent 726e66ea, child 0443cef8, origin xyz=-0.0132225166836 0.0 0.0 rpy=0 0 0, axis 0 1 0, limit lower=-1.9 upper=0.31033780141 effort=0.966661265437 velocity=0.375509633371
- added joint 7890965f7d2f91e4: type revolute, parent 7890965f, child 7d2f91e4, origin xyz=0.0 -0.0227442211358 0.0 rpy=0 0 0, axis 0 1 0, limit lower=-1.9 upper=0.965562611806 effort=0.456445009719 velocity=0.496143208028
- added joint 7d2f91e483cccbd2: type revolute, parent 7d2f91e4, child 83cccbd2, origin xyz=0.0 -0.107914655121 0.0 rpy=0 0 0, axis 0 0 1, limit lower=-1.9 upper=0.136554408429 effort=1.16324054574 velocity=0.312047690829
- added joint 83cccbd29b5bd92e: type revolute, parent 83cccbd2, child 9b5bd92e, origin xyz=-0.0724202115472 0.0 0.0 rpy=0 0 0, axis 0 0 1, limit lower=-1.9 upper=0.546211899938 effort=1.61402201093 velocity=0.41306019182
- added joint 85decfd814945161: type revolute, parent 85decfd8, child 14945161, origin xyz=0.0610886104192 0.0 0.0 rpy=0 0 0, axis 0 1 0, limit lower=-1.9 upper=0.102064901649 effort=0.422151747483 velocity=0.0450838143262
- added joint 87d7940f3da6150c: type revolute, parent 87d7940f, child 3da6150c, origin xyz=0.0 -0.0444796676004 0.0 rpy=0 0 0, axis 0 0 1, limit lower=-1.9 upper=0.108436483346 effort=0.248115820582 velocity=0.0432701746453
- added joint 954daca0982855a3: type revolute, parent 954daca0, child 982855a3, origin xyz=0.0 0.115377989296 0.0 rpy=0 0 0, axis 0 0 1, limit lower=-1.9 upper=1.9 effort=0.923371919085 velocity=0.350787041946
- added joint 982855a3726e66ea: type revolute, parent 982855a3, child 726e66ea, origin xyz=0.0 0.0 -0.0154031405075 rpy=0 0 0, axis 0 0 1, limit lower=-1.9 upper=0.947139027845 effort=0.590223233034 velocity=0.673824204898
- added joint 9b5bd92e64c6f495: type revolute, parent 9b5bd92e, child 64c6f495, origin xyz=0.0 -0.067132646337 0.0 rpy=0 0 0, axis 0 0 1, limit lower=-1.9 upper=0.0270449108059 effort=0.467977716796 velocity=0.0667382953089
- added joint 9cdb5009954daca0: type revolute, parent 9cdb5009, child 954daca0, origin xyz=0.0 -0.0677195858122 0.0 rpy=0 0 0, axis 0 0 1, limit lower=-1.9 upper=0.341737776897 effort=0.286404521279 velocity=1.05138691724
- added joint b51909636ec480c8: type revolute, parent b5190963, child 6ec480c8, origin xyz=0.0 0.296890064168 0.0 rpy=0 0 0, axis 0 0 1, limit lower=-1.9 upper=0.0379795368137 effort=0.376926836267 velocity=0.117704652072
- added joint c9507b8b3691be7d: type revolute, parent c9507b8b, child 3691be7d, origin xyz=0.0 0.0 -0.0450365789612 rpy=0 0 0, axis 0 0 1, limit lower=-1.9 upper=0.379670717296 effort=0.0489190980108 velocity=0.358481678273
- added joint d63c789b413041c7: type revolute, parent d63c789b, child 413041c7, origin xyz=0.0 0.0184764451506 0.0 rpy=0 0 0, axis 0 0 1, limit lower=-1.9 upper=0.169053180115 effort=0.0562923070372 velocity=0.495129841063
- added joint d78aac32105cdbe8: type revolute, parent d78aac32, child 105cdbe8, origin xyz=0.0 0.236723511144 0.0 rpy=0 0 0, axis 0 0 1, limit lower=-1.9 upper=0.29564136956 effort=0.729112972127 velocity=0.155432521834
- added joint e68ff6a405fb6450: type revolute, parent e68ff6a4, child 05fb6450, origin xyz=0.0 -0.160221870822 0.0 rpy=0 0 0, axis 0 0 1, limit lower=-1.9 upper=0.28871898528 effort=0.952429653087 velocity=0.482212154929
- added joint e8e5e8db85decfd8: type revolute, parent e8e5e8db, child 85decfd8, origin xyz=0.0 0.0 -0.125876742615 rpy=0 0 0, axis 0 1 0, limit lower=-1.9 upper=1.039609111 effort=0.274750256226 velocity=0.786927801371
- added joint ea98e739b5190963: type revolute, parent ea98e739, child b5190963, origin xyz=-0.0501145990306 0.0 0.0 rpy=0 0 0, axis 0 0 1, limit lower=-1.9 upper=0.837651867618 effort=0.93982556605 velocity=0.412559300874
- added joint f3d7be28e8e5e8db: type revolute, parent f3d7be28, child e8e5e8db, origin xyz=0.0 -0.0764411391882 0.0 rpy=0 0 0, axis 0 0 1, limit lower=-1.9 upper=0.40624931156 effort=2.69866842273 velocity=0.0557960429855
