Commit message: Tweaking mutation parameters

File: robot.urdf (robot description, URDF)
Before this commit: robot paul, 40 links, 39 joints
Links:
- removed link 0443cef8
- removed link 05fb6450
- removed link 0b5a6eef
- removed link 0cdc028b
- removed link 0f457723
- removed link 105cdbe8
- removed link 14945161
- removed link 18b29c49
- removed link 275c27f4
- removed link 30fc0f2e
- removed link 3156b1b7
- removed link 3691be7d
- removed link 377fa558
- removed link 3da6150c
- removed link 413041c7
- removed link 4b7a5ff1
- removed link 591f5e18
- removed link 64c6f495
- removed link 6842db81
- removed link 6ec480c8
- removed link 70a813a7
- removed link 726e66ea
- removed link 7890965f
- removed link 7d2f91e4
- removed link 83cccbd2
- removed link 85decfd8
- removed link 87d7940f
- removed link 954daca0
- removed link 982855a3
- removed link 9b5bd92e
- removed link 9cdb5009
- removed link b5190963
- removed link bb90fee0
- removed link c9507b8b
- removed link d63c789b
- removed link d78aac32
- removed link e68ff6a4
- removed link e8e5e8db
- removed link ea98e739
- removed link f3d7be28
- added link 15183ac2, mass 0.002765209452; collision box size=0.0114284594376 0.0193991582252 0.099780906054; visual box size=0.0114284594376 0.0193991582252 0.099780906054
- added link 29907e43, mass 0.00136928967617; collision box size=0.0145291784676 0.0120034111686 0.0628115599706; visual box size=0.0145291784676 0.0120034111686 0.0628115599706
- added link 56c25184, mass 16.8068077994; collision box size=0.164163330301 0.0557477243164 14.6916956498; visual box size=0.164163330301 0.0557477243164 14.6916956498
Joints:
- removed joint 0443cef8591f5e18
- removed joint 05fb645087d7940f
- removed joint 0b5a6eefea98e739
- removed joint 0cdc028bbb90fee0
- removed joint 0f4577236842db81
- removed joint 105cdbe89cdb5009
- removed joint 14945161377fa558
- removed joint 18b29c49f3d7be28
- removed joint 275c27f4d78aac32
- removed joint 30fc0f2e3156b1b7
- removed joint 3156b1b718b29c49
- removed joint 3691be7d30fc0f2e
- removed joint 377fa5584b7a5ff1
- removed joint 3da6150c70a813a7
- removed joint 413041c7e68ff6a4
- removed joint 4b7a5ff10b5a6eef
- removed joint 591f5e180cdc028b
- removed joint 64c6f495275c27f4
- removed joint 6842db81c9507b8b
- removed joint 6ec480c8d63c789b
- removed joint 70a813a77890965f
- removed joint 726e66ea0443cef8
- removed joint 7890965f7d2f91e4
- removed joint 7d2f91e483cccbd2
- removed joint 83cccbd29b5bd92e
- removed joint 85decfd814945161
- removed joint 87d7940f3da6150c
- removed joint 954daca0982855a3
- removed joint 982855a3726e66ea
- removed joint 9b5bd92e64c6f495
- removed joint 9cdb5009954daca0
- removed joint b51909636ec480c8
- removed joint c9507b8b3691be7d
- removed joint d63c789b413041c7
- removed joint d78aac32105cdbe8
- removed joint e68ff6a405fb6450
- removed joint e8e5e8db85decfd8
- removed joint ea98e739b5190963
- removed joint f3d7be28e8e5e8db
- added joint 29907e4356c25184: type revolute, parent 29907e43, child 56c25184, origin xyz=0.0 0.0 -14.6916956498 rpy=0 0 0, axis 0 0 1, limit lower=-1.9 upper=0.414710442446 effort=0.420992724841 velocity=0.275109006267
- added joint 56c2518415183ac2: type revolute, parent 56c25184, child 15183ac2, origin xyz=0.0 0.0 -0.099780906054 rpy=0 0 0, axis 1 0 0, limit lower=-1.9 upper=1.9 effort=0 velocity=0

Commit message: Adding tests

File: robot.urdf (robot description, URDF)
Before this commit: robot paul, 3 links, 2 joints
Links:
- removed link 15183ac2
- removed link 29907e43
- removed link 56c25184
- added link 1df380c7, mass 0.108564482391; collision box size=0.074722514903 0.253503821318 0.0458502557502; visual box size=0.074722514903 0.253503821318 0.0458502557502
- added link 2d120c78, mass 0.0181777393763; collision box size=0.0495142872232 0.0478916143612 0.0613253239522; visual box size=0.0495142872232 0.0478916143612 0.0613253239522
- added link 7ec90f42, mass 0.00737896833999; collision box size=0.0181899311883 0.143242268628 0.0226560078872; visual box size=0.0181899311883 0.143242268628 0.0226560078872
Joints:
- removed joint 29907e4356c25184
- removed joint 56c2518415183ac2
- added joint 1df380c77ec90f42: type revolute, parent 1df380c7, child 7ec90f42, origin xyz=-0.0181899311883 0.0 0.0 rpy=0 0 0, axis 0 0 1, limit lower=-1.9 upper=0.305980647752 effort=0.340390795 velocity=0.8254399068
- added joint 2d120c781df380c7: type revolute, parent 2d120c78, child 1df380c7, origin xyz=0.0 0.0 0.0458502557502 rpy=0 0 0, axis 0 1 0, limit lower=-1.9 upper=0.118973038075 effort=0.622476191893 velocity=0.381694569133

Commit message: Adding more unit tests

File: robot.urdf (robot description, URDF)
Before this commit: robot paul, 3 links, 2 joints
Links:
- removed link 1df380c7
- removed link 2d120c78
- removed link 7ec90f42
- added link c697baa6, mass 1; collision box size=0.2 0.2 0.2; visual box size=0.2 0.2 0.2
Joints:
- removed joint 1df380c77ec90f42
- removed joint 2d120c781df380c7
